Commit message: Renamed joint0, joint1 to left and right wheel joints

File: ros/src/odrive_description/urdf/odrive.ros2_control.xacro (robot description, xacro)
@@ -1,11 +1,11 @@
 <?xml version="1.0"?>
 <robot xmlns:xacro="http://www.ros.org/wiki/xacro">
-  <xacro:macro name="odrive_ros2_control" params="name enable_joint0:=^|true enable_joint1:=^|true">
+  <xacro:macro name="odrive_ros2_control" params="name enable_left_wheel_joint:=^|true enable_right_wheel_joint:=^|true">
     <ros2_control name="${name}" type="system">
       <hardware>
         <plugin>odrive_hardware_interface/ODriveHardwareInterface</plugin>
       </hardware>
-      <xacro:if value="${enable_joint0}">
-        <joint name="joint0">
+      <xacro:if value="${enable_left_wheel_joint}">
+        <joint name="left_wheel_joint">
           <command_interface  name="position" />
           <command_interface  name="velocity" />
@@ -27,6 +27,6 @@
         </sensor>
       </xacro:if>
-      <xacro:if value="${enable_joint1}">
-        <joint name="joint1">
+      <xacro:if value="${enable_right_wheel_joint}">
+        <joint name="right_wheel_joint">
           <command_interface  name="position" />
           <command_interface  name="velocity" />

File: ros/src/odrive_description/urdf/odrive.urdf.xacro (robot description, xacro)
@@ -1,11 +1,11 @@
 <?xml version="1.0"?>
 <robot xmlns:xacro="http://www.ros.org/wiki/xacro" name="odrive">
-  <xacro:arg name="enable_joint0" default="true" />
-  <xacro:arg name="enable_joint1" default="true" />
+  <xacro:arg name="enable_left_wheel_joint" default="true" />
+  <xacro:arg name="enable_right_wheel_joint" default="true" />
   <xacro:include filename="$(find odrive_description)/urdf/odrive.ros2_control.xacro" />
   <link name="world" />
-  <xacro:if value="$(arg enable_joint0)">
+  <xacro:if value="$(arg enable_left_wheel_joint)">
     <link name="link0" />
-    <joint name="joint0" type="continuous">
+    <joint name="left_wheel_joint" type="continuous">
       <parent link="world"/>
       <child link="link0"/>
@@ -13,7 +13,7 @@
     </joint>
   </xacro:if>
-  <xacro:if value="$(arg enable_joint1)">
+  <xacro:if value="$(arg enable_right_wheel_joint)">
     <link name="link1" />
-    <joint name="joint1" type="continuous">
+    <joint name="right_wheel_joint" type="continuous">
       <parent link="world"/>
       <child link="link1"/>
@@ -23,5 +23,5 @@
   <xacro:odrive_ros2_control
     name="odrive_ros2_control"
-    enable_joint0="$(arg enable_joint0)"
-    enable_joint1="$(arg enable_joint1)" />
+    enable_left_wheel_joint="$(arg enable_left_wheel_joint)"
+    enable_right_wheel_joint="$(arg enable_right_wheel_joint)" />
 </robot>
