Commit message: Working on rosbot odrive hardware

File: ros/src/rosbot_description/ros2_control/rosbot_system.ros2_control.xacro (robot description, xacro)
@@ -10,26 +10,75 @@
         </xacro:if>
         <xacro:unless value="${use_fake_hardware}">
+          <!--
           <plugin>ros2_control_demo_hardware/DiffBotSystemHardware</plugin>
           <param name="example_param_hw_start_duration_sec">2.0</param>
           <param name="example_param_hw_stop_duration_sec">3.0</param>
-        </xacro:unless>
-      </hardware>
-      <joint name="left_wheel_joint">
-        <command_interface name="velocity">
-          <param name="min">-1</param>
-          <param name="max">1</param>
-        </command_interface>
-        <state_interface name="position"/>
-        <state_interface name="velocity"/>
-      </joint>
-      <joint name="right_wheel_joint">
-        <command_interface name="velocity">
-          <param name="min">-1</param>
-          <param name="max">1</param>
-        </command_interface>
-        <state_interface name="position"/>
-        <state_interface name="velocity"/>
-      </joint>
-    </ros2_control>
-  </xacro:macro>
+           -->
+          <!-- <hardware> -->
+          <plugin>odrive_hardware_interface/ODriveHardwareInterface</plugin>
+          <!-- </hardware> -->
+          <!-- TODO: move out of <hardware/>? -->
+          <!-- <xacro:if value="${enable_left_wheel_joint}"> -->
+          <joint name="left_wheel_joint">
+            <command_interface name="position" />
+            <command_interface name="velocity" />
+            <command_interface name="effort" />
+            <state_interface name="position" />
+            <state_interface name="velocity" />
+            <state_interface name="effort" />
+            <param name="axis">0</param>
+            <param name="enable_watchdog">1</param>
+            <param name="watchdog_timeout">0.1</param>
+          </joint>
+          <sensor name="axis0">
+            <state_interface name="axis_error" />
+            <state_interface name="motor_error" />
+            <state_interface name="encoder_error" />
+            <state_interface name="controller_error" />
+            <state_interface name="fet_temperature" />
+            <state_interface name="motor_temperature" />
+          </sensor>
+          <!-- </xacro:if> -->
+          <!-- <xacro:if value="${enable_right_wheel_joint}"> -->
+          <joint name="right_wheel_joint">
+            <command_interface name="position" />
+            <command_interface name="velocity" />
+            <command_interface name="effort" />
+            <state_interface name="position" />
+            <state_interface name="velocity" />
+            <state_interface name="effort" />
+            <param name="axis">1</param>
+            <param name="enable_watchdog">1</param>
+            <param name="watchdog_timeout">0.1</param>
+          </joint>
+          <sensor name="axis1">
+            <state_interface name="axis_error" />
+            <state_interface name="motor_error" />
+            <state_interface name="encoder_error" />
+            <state_interface name="controller_error" />
+            <state_interface name="fet_temperature" />
+            <state_interface name="motor_temperature" />
+          </sensor>
+          <!-- </xacro:if> -->
+        </ros2_control>
+      </xacro:unless>
+    </hardware>
+    <joint name="left_wheel_joint">
+      <command_interface name="velocity">
+        <param name="min">-1</param>
+        <param name="max">1</param>
+      </command_interface>
+      <state_interface name="position"/>
+      <state_interface name="velocity"/>
+    </joint>
+    <joint name="right_wheel_joint">
+      <command_interface name="velocity">
+        <param name="min">-1</param>
+        <param name="max">1</param>
+      </command_interface>
+      <state_interface name="position"/>
+      <state_interface name="velocity"/>
+    </joint>
+  </ros2_control>
+</xacro:macro>
 </robot>

File: ros/src/rosbot_description/urdf/rosbot.urdf.xacro (robot description, xacro)
@@ -1,3 +1,5 @@
 <?xml version="1.0"?>
+<!-- TODO: add name here? -->
+<!-- <robot xmlns:xacro="http://www.ros.org/wiki/xacro" name="rosbot"> -->
 <robot xmlns:xacro="http://www.ros.org/wiki/xacro">
   <xacro:macro name="rosbot" params="prefix">

Commit message: Working on rosbot urdf

File: ros/src/rosbot_description/ros2_control/rosbot_system.ros2_control.xacro (robot description, xacro)
@@ -20,5 +20,5 @@
           <!-- TODO: move out of <hardware/>? -->
           <!-- <xacro:if value="${enable_left_wheel_joint}"> -->
-          <joint name="left_wheel_joint">
+          <!-- <joint name="left_wheel_joint">
             <command_interface name="position" />
             <command_interface name="velocity" />
@@ -38,8 +38,8 @@
             <state_interface name="fet_temperature" />
             <state_interface name="motor_temperature" />
-          </sensor>
+          </sensor> -->
           <!-- </xacro:if> -->
           <!-- <xacro:if value="${enable_right_wheel_joint}"> -->
-          <joint name="right_wheel_joint">
+          <!-- <joint name="right_wheel_joint">
             <command_interface name="position" />
             <command_interface name="velocity" />
@@ -59,5 +59,5 @@
             <state_interface name="fet_temperature" />
             <state_interface name="motor_temperature" />
-          </sensor>
+          </sensor> -->
           <!-- </xacro:if> -->
         </ros2_control>
@@ -71,4 +71,5 @@
       <state_interface name="position"/>
       <state_interface name="velocity"/>
+      <!-- TODO: add extra joint interfaces, state from above? -->
     </joint>
     <joint name="right_wheel_joint">

Commit message: Fixed urdf issue

File: ros/src/rosbot_description/ros2_control/rosbot_system.ros2_control.xacro (robot description, xacro)
@@ -61,25 +61,24 @@
           </sensor> -->
           <!-- </xacro:if> -->
-        </ros2_control>
-      </xacro:unless>
-    </hardware>
-    <joint name="left_wheel_joint">
-      <command_interface name="velocity">
-        <param name="min">-1</param>
-        <param name="max">1</param>
-      </command_interface>
-      <state_interface name="position"/>
-      <state_interface name="velocity"/>
-      <!-- TODO: add extra joint interfaces, state from above? -->
-    </joint>
-    <joint name="right_wheel_joint">
-      <command_interface name="velocity">
-        <param name="min">-1</param>
-        <param name="max">1</param>
-      </command_interface>
-      <state_interface name="position"/>
-      <state_interface name="velocity"/>
-    </joint>
-  </ros2_control>
-</xacro:macro>
+        </xacro:unless>
+      </hardware>
+      <joint name="left_wheel_joint">
+        <command_interface name="velocity">
+          <param name="min">-1</param>
+          <param name="max">1</param>
+        </command_interface>
+        <state_interface name="position"/>
+        <state_interface name="velocity"/>
+        <!-- TODO: add extra joint interfaces, state from above? -->
+      </joint>
+      <joint name="right_wheel_joint">
+        <command_interface name="velocity">
+          <param name="min">-1</param>
+          <param name="max">1</param>
+        </command_interface>
+        <state_interface name="position"/>
+        <state_interface name="velocity"/>
+      </joint>
+    </ros2_control>
+  </xacro:macro>
 </robot>

Commit message: Removed enable left/right wheel joint arguments

File: ros/src/rosbot_description/ros2_control/rosbot_system.ros2_control.xacro (robot description, xacro)
@@ -10,55 +10,5 @@
         </xacro:if>
         <xacro:unless value="${use_fake_hardware}">
-          <!--
-          <plugin>ros2_control_demo_hardware/DiffBotSystemHardware</plugin>
-          <param name="example_param_hw_start_duration_sec">2.0</param>
-          <param name="example_param_hw_stop_duration_sec">3.0</param>
-           -->
-          <!-- <hardware> -->
           <plugin>odrive_hardware_interface/ODriveHardwareInterface</plugin>
-          <!-- </hardware> -->
-          <!-- TODO move out of <hardware/>? -->
-          <!-- <xacro:if value="${enable_left_wheel_joint}"> -->
-          <!-- <joint name="left_wheel_joint">
-            <command_interface name="position" />
-            <command_interface name="velocity" />
-            <command_interface name="effort" />
-            <state_interface name="position" />
-            <state_interface name="velocity" />
-            <state_interface name="effort" />
-            <param name="axis">0</param>
-            <param name="enable_watchdog">1</param>
-            <param name="watchdog_timeout">0.1</param>
-          </joint>
-          <sensor name="axis0">
-            <state_interface name="axis_error" />
-            <state_interface name="motor_error" />
-            <state_interface name="encoder_error" />
-            <state_interface name="controller_error" />
-            <state_interface name="fet_temperature" />
-            <state_interface name="motor_temperature" />
-          </sensor> -->
-          <!-- </xacro:if> -->
-          <!-- <xacro:if value="${enable_right_wheel_joint}"> -->
-          <!-- <joint name="right_wheel_joint">
-            <command_interface name="position" />
-            <command_interface name="velocity" />
-            <command_interface name="effort" />
-            <state_interface name="position" />
-            <state_interface name="velocity" />
-            <state_interface name="effort" />
-            <param name="axis">1</param>
-            <param name="enable_watchdog">1</param>
-            <param name="watchdog_timeout">0.1</param>
-          </joint>
-          <sensor name="axis1">
-            <state_interface name="axis_error" />
-            <state_interface name="motor_error" />
-            <state_interface name="encoder_error" />
-            <state_interface name="controller_error" />
-            <state_interface name="fet_temperature" />
-            <state_interface name="motor_temperature" />
-          </sensor> -->
-          <!-- </xacro:if> -->
         </xacro:unless>
       </hardware>

Commit message: Added rviz transform

File: ros/src/rosbot_description/ros2_control/rosbot_system.ros2_control.xacro (robot description, xacro)
@@ -25,5 +25,5 @@
         <param name="axis">0</param>
         <param name="enable_watchdog">1</param>
-        <param name="watchdog_timeout">0.2</param>
+        <param name="watchdog_timeout">0.5</param>
       </joint>
       <sensor name="axis0">
@@ -47,5 +47,5 @@
         <param name="axis">1</param>
         <param name="enable_watchdog">1</param>
-        <param name="watchdog_timeout">0.2</param>
+        <param name="watchdog_timeout">0.5</param>
       </joint>
       <sensor name="axis1">

File: ros/src/rosbot_description/urdf/rosbot.urdf.xacro (robot description, xacro)
@@ -135,10 +135,10 @@
       <parent link="${prefix}base_link"/>
       <child link="${prefix}lidar"/>
-      <origin xyz="0 0 ${body_height/2 + lidar_height/2}" rpy="0 0 0"/>
+      <origin xyz="${-rear_wheels_axis_offset} 0 ${body_height/2 + lidar_height/2}" rpy="0 0 0"/>
       <axis xyz="0 0 1"/>
     </joint>
     <link name="${prefix}lidar">
       <visual>
-        <origin xyz="0 0 ${body_height/2 + lidar_height/2}" rpy="0 0 0"/>
+        <origin xyz="${-rear_wheels_axis_offset} 0 ${body_height/2 + lidar_height/2}" rpy="0 0 0"/>
         <geometry>
           <box size="${lidar_width} ${lidar_length} ${lidar_height}"/>
