Commit message: Updated robot dimensions in urdf

File: ros/src/rosbot_description/urdf/rosbot.urdf.xacro (robot description, xacro)
@@ -6,18 +6,30 @@
     <!-- Constants for robot dimensions -->
     <xacro:property name="PI" value="3.1415926535897931"/>
-    <xacro:property name="base_mass" value="0.3" />
+    <xacro:property name="base_mass" value="6.0" />
     <!-- arbitrary value for base mass -->
-    <xacro:property name="base_width" value="0.1" />
-    <xacro:property name="base_length" value="0.1" />
-    <xacro:property name="base_height" value="0.05" />
-    <xacro:property name="wheel_mass" value="0.3" />
+    <xacro:property name="base_width" value="0.3" />
+    <xacro:property name="base_length" value="0.46" />
+    <xacro:property name="base_height" value="0.17" />
+    <xacro:property name="wheel_mass" value="0.5" />
     <!-- arbitrary value for wheel mass -->
-    <xacro:property name="wheel_len" value="0.020" />
-    <xacro:property name="wheel_radius" value="0.015" />
+    <xacro:property name="wheel_len" value="0.05" />
+    <xacro:property name="wheel_radius" value="0.195" />
     <xacro:property name="caster_wheel_mass" value="0.1" />
     <!-- arbitrary value for caster wheel mass -->
     <xacro:property name="caster_wheel_radius" value="0.015" />
-    <xacro:property name="z_offset" value="-${base_height/2}" />
+    <!-- <xacro:property name="z_offset" value="-${base_height/2}" /> -->
+    <xacro:property name="z_offset" value="-0.0975" />
     <!-- Space btw top of beam and the each joint -->
+    <!-- robot is 300mm wide, 460mm long, 170mm tall -->
+    <!-- front wheels are 38.5mm off the ground surface -->
+    <!-- robot body is 57.5mm off the ground surface -->
+    <!-- robot rear wheel radius is 195mm -->
+    <!-- robot rear wheels axis is 97.5mm off the ground surface -->
+    <!-- robot rear wheels axis is 100mm from the center of the body -->
+    <!-- front wheel radius 77mm  -->
+    <!-- robot front wheels axis is -267.57mm from the center of the body -->
+    <!-- small motor pulley has 16 teeth -->
+    <!-- large wheel pulley has 72 teeth -->
+    <!-- motor to wheel gear ratio is 72/16 = 4.5 -->
     <!-- Base Link -->
     <link name="${prefix}base_link">

Commit message: Added rviz and teleop launch scripts, removed caster wheels

File: ros/src/rosbot_description/urdf/rosbot.urdf.xacro (robot description, xacro)
@@ -15,7 +15,4 @@
     <xacro:property name="wheel_len" value="0.05" />
     <xacro:property name="wheel_radius" value="0.195" />
-    <xacro:property name="caster_wheel_mass" value="0.1" />
-    <!-- arbitrary value for caster wheel mass -->
-    <xacro:property name="caster_wheel_radius" value="0.015" />
     <!-- <xacro:property name="z_offset" value="-${base_height/2}" /> -->
     <xacro:property name="z_offset" value="-0.0975" />
@@ -109,56 +106,4 @@
       </inertial>
     </link>
-    <joint name="${prefix}caster_frontal_wheel_joint" type="fixed">
-      <parent link="${prefix}base_link"/>
-      <child link="${prefix}caster_frontal_wheel"/>
-      <origin xyz="${base_width/2 - caster_wheel_radius} 0 ${z_offset}" rpy="0 0 0"/>
-    </joint>
-    <!-- caster frontal wheel Link -->
-    <link name="${prefix}caster_frontal_wheel">
-      <collision>
-        <origin xyz="0 0 0" rpy="0 0 0"/>
-        <geometry>
-          <sphere radius="${caster_wheel_radius}"/>
-        </geometry>
-      </collision>
-      <visual>
-        <origin xyz="0 0 0" rpy="0 0 0"/>
-        <geometry>
-          <sphere radius="${caster_wheel_radius}"/>
-        </geometry>
-        <material name="white"/>
-      </visual>
-      <inertial>
-        <origin xyz="0 0 0" rpy="0 0 0"/>
-        <mass value="${caster_wheel_mass}"/>
-        <inertia ixx="${caster_wheel_mass * 0.4 * (caster_wheel_radius * caster_wheel_radius)}" ixy="0.0" ixz="0.0" iyy="${caster_wheel_mass * 0.4 * (caster_wheel_radius * caster_wheel_radius)}" iyz="0.0" izz="${caster_wheel_mass * 0.4 * (caster_wheel_radius * caster_wheel_radius)}"/>
-      </inertial>
-    </link>
-    <joint name="${prefix}caster_rear_wheel_joint" type="fixed">
-      <parent link="${prefix}base_link"/>
-      <child link="${prefix}caster_rear_wheel"/>
-      <origin xyz="${-base_width/2 + caster_wheel_radius} 0 ${z_offset}" rpy="0 0 0"/>
-    </joint>
-    <!-- caster rear wheel Link -->
-    <link name="${prefix}caster_rear_wheel">
-      <collision>
-        <origin xyz="0 0 0" rpy="0 0 0"/>
-        <geometry>
-          <sphere radius="${caster_wheel_radius}"/>
-        </geometry>
-      </collision>
-      <visual>
-        <origin xyz="0 0 0" rpy="0 0 0"/>
-        <geometry>
-          <sphere radius="${caster_wheel_radius}"/>
-        </geometry>
-        <material name="white"/>
-      </visual>
-      <inertial>
-        <origin xyz="0 0 0" rpy="0 0 0"/>
-        <mass value="${caster_wheel_mass}"/>
-        <inertia ixx="${caster_wheel_mass * 0.4 * (caster_wheel_radius * caster_wheel_radius)}" ixy="0.0" ixz="0.0" iyy="${caster_wheel_mass * 0.4 * (caster_wheel_radius * caster_wheel_radius)}" iyz="0.0" izz="${caster_wheel_mass * 0.4 * (caster_wheel_radius * caster_wheel_radius)}"/>
-      </inertial>
-    </link>
   </xacro:macro>
 </robot>

Commit message: Updated robot rviz dimensions

File: ros/src/rosbot_description/urdf/rosbot.urdf.xacro (robot description, xacro)
@@ -8,11 +8,11 @@
     <xacro:property name="base_mass" value="6.0" />
     <!-- arbitrary value for base mass -->
-    <xacro:property name="base_width" value="0.3" />
-    <xacro:property name="base_length" value="0.46" />
+    <xacro:property name="base_width" value="0.46" />
+    <xacro:property name="base_length" value="0.3" />
     <xacro:property name="base_height" value="0.17" />
     <xacro:property name="wheel_mass" value="0.5" />
     <!-- arbitrary value for wheel mass -->
     <xacro:property name="wheel_len" value="0.05" />
-    <xacro:property name="wheel_radius" value="0.195" />
+    <xacro:property name="wheel_radius" value="0.0975" />
     <!-- <xacro:property name="z_offset" value="-${base_height/2}" /> -->
     <xacro:property name="z_offset" value="-0.0975" />
@@ -21,5 +21,5 @@
     <!-- front wheels are 38.5mm off the ground surface -->
     <!-- robot body is 57.5mm off the ground surface -->
-    <!-- robot rear wheel radius is 195mm -->
+    <!-- robot rear wheel diameter is 195mm (radius 97.5mm) -->
     <!-- robot rear wheels axis is 97.5mm off the ground surface -->
     <!-- robot rear wheels axis is 100mm from the center of the body -->

Commit message: Working on robot rviz parameters

File: ros/src/rosbot_description/urdf/rosbot.urdf.xacro (robot description, xacro)
@@ -15,6 +15,7 @@
     <xacro:property name="wheel_len" value="0.05" />
     <xacro:property name="wheel_radius" value="0.0975" />
-    <!-- <xacro:property name="z_offset" value="-${base_height/2}" /> -->
-    <xacro:property name="z_offset" value="-0.0975" />
+    <xacro:property name="rear_wheel_ground_offset" value="0.0975" />
+    <xacro:property name="rear_wheels_axis_offset" value="0.1" />
+    <xacro:property name="rear_wheels_distance" value="0.24" />
     <!-- Space btw top of beam and the each joint -->
     <!-- robot is 300mm wide, 460mm long, 170mm tall -->
@@ -53,5 +54,5 @@
       <parent link="${prefix}base_link"/>
       <child link="${prefix}left_wheel"/>
-      <origin xyz="0 -${base_width/2} ${z_offset}" rpy="0 0 0"/>
+      <origin xyz="-${rear_wheels_axis_offset} -${rear_wheels_distance/2} ${rear_wheel_ground_offset}" rpy="0 0 0"/>
       <axis xyz="0 1 0"/>
       <dynamics damping="0.2"/>
@@ -81,5 +82,5 @@
       <parent link="${prefix}base_link"/>
       <child link="${prefix}right_wheel"/>
-      <origin xyz="0 ${base_width/2} ${z_offset}" rpy="0 0 0"/>
+      <origin xyz="-${rear_wheels_axis_offset} ${rear_wheels_distance/2} ${rear_wheel_ground_offset}" rpy="0 0 0"/>
       <axis xyz="0 1 0"/>
       <dynamics damping="0.2"/>

Commit message: Working on robot rviz parameters 2

File: ros/src/rosbot_description/urdf/rosbot.urdf.xacro (robot description, xacro)
@@ -15,7 +15,8 @@
     <xacro:property name="wheel_len" value="0.05" />
     <xacro:property name="wheel_radius" value="0.0975" />
+    <xacro:property name="frame_ground_offset" value="0.0575" />
     <xacro:property name="rear_wheel_ground_offset" value="0.0975" />
     <xacro:property name="rear_wheels_axis_offset" value="0.1" />
-    <xacro:property name="rear_wheels_distance" value="0.24" />
+    <xacro:property name="rear_wheels_distance" value="0.2476" />
     <!-- Space btw top of beam and the each joint -->
     <!-- robot is 300mm wide, 460mm long, 170mm tall -->
@@ -33,5 +34,5 @@
     <link name="${prefix}base_link">
       <collision>
-        <origin xyz="0 0 0" rpy="0 0 0"/>
+        <origin xyz="0 0 ${frame_ground_offset}" rpy="0 0 0"/>
         <geometry>
           <box size="${base_width} ${base_length} ${base_height}"/>
@@ -39,5 +40,5 @@
       </collision>
       <visual>
-        <origin xyz="0 0 0" rpy="0 0 0"/>
+        <origin xyz="0 0 ${frame_ground_offset}" rpy="0 0 0"/>
         <geometry>
           <box size="${base_width} ${base_length} ${base_height}"/>
@@ -46,5 +47,5 @@
       </visual>
       <inertial>
-        <origin xyz="0 0 0" rpy="0 0 0"/>
+        <origin xyz="0 0 ${frame_ground_offset}" rpy="0 0 0"/>
         <mass value="${base_mass}"/>
         <inertia ixx="${base_mass / 12.0 * (base_length*base_length + base_height*base_height)}" ixy="0.0" ixz="0.0" iyy="${base_mass / 12.0 * (base_height*base_height + base_width*base_width)}" iyz="0.0" izz="${base_mass / 12.0 * (base_width*base_width + base_length*base_length)}"/>

Commit message: Working on robot rviz parameters 3

File: ros/src/rosbot_description/urdf/rosbot.urdf.xacro (robot description, xacro)
@@ -34,5 +34,5 @@
     <link name="${prefix}base_link">
       <collision>
-        <origin xyz="0 0 ${frame_ground_offset}" rpy="0 0 0"/>
+        <origin xyz="0 0 ${base_height/2 + frame_ground_offset}" rpy="0 0 0"/>
         <geometry>
           <box size="${base_width} ${base_length} ${base_height}"/>
@@ -40,5 +40,5 @@
       </collision>
       <visual>
-        <origin xyz="0 0 ${frame_ground_offset}" rpy="0 0 0"/>
+        <origin xyz="0 0 ${base_height/2 + frame_ground_offset}" rpy="0 0 0"/>
         <geometry>
           <box size="${base_width} ${base_length} ${base_height}"/>
@@ -47,5 +47,5 @@
       </visual>
       <inertial>
-        <origin xyz="0 0 ${frame_ground_offset}" rpy="0 0 0"/>
+        <origin xyz="0 0 ${base_height/2 + frame_ground_offset}" rpy="0 0 0"/>
         <mass value="${base_mass}"/>
         <inertia ixx="${base_mass / 12.0 * (base_length*base_length + base_height*base_height)}" ixy="0.0" ixz="0.0" iyy="${base_mass / 12.0 * (base_height*base_height + base_width*base_width)}" iyz="0.0" izz="${base_mass / 12.0 * (base_width*base_width + base_length*base_length)}"/>

Commit message: Replaced wheel offset with body offset

File: ros/src/rosbot_description/urdf/rosbot.urdf.xacro (robot description, xacro)
@@ -34,5 +34,5 @@
     <link name="${prefix}base_link">
       <collision>
-        <origin xyz="0 0 ${base_height/2 + frame_ground_offset}" rpy="0 0 0"/>
+        <origin xyz="${rear_wheels_axis_offset} 0 ${base_height/2 + frame_ground_offset}" rpy="0 0 0"/>
         <geometry>
           <box size="${base_width} ${base_length} ${base_height}"/>
@@ -40,5 +40,5 @@
       </collision>
       <visual>
-        <origin xyz="0 0 ${base_height/2 + frame_ground_offset}" rpy="0 0 0"/>
+        <origin xyz="${rear_wheels_axis_offset} 0 ${base_height/2 + frame_ground_offset}" rpy="0 0 0"/>
         <geometry>
           <box size="${base_width} ${base_length} ${base_height}"/>
@@ -47,5 +47,5 @@
       </visual>
       <inertial>
-        <origin xyz="0 0 ${base_height/2 + frame_ground_offset}" rpy="0 0 0"/>
+        <origin xyz="${rear_wheels_axis_offset} 0 ${base_height/2 + frame_ground_offset}" rpy="0 0 0"/>
         <mass value="${base_mass}"/>
         <inertia ixx="${base_mass / 12.0 * (base_length*base_length + base_height*base_height)}" ixy="0.0" ixz="0.0" iyy="${base_mass / 12.0 * (base_height*base_height + base_width*base_width)}" iyz="0.0" izz="${base_mass / 12.0 * (base_width*base_width + base_length*base_length)}"/>
@@ -55,5 +55,5 @@
       <parent link="${prefix}base_link"/>
       <child link="${prefix}left_wheel"/>
-      <origin xyz="-${rear_wheels_axis_offset} -${rear_wheels_distance/2} ${rear_wheel_ground_offset}" rpy="0 0 0"/>
+      <origin xyz="0 -${rear_wheels_distance/2} ${rear_wheel_ground_offset}" rpy="0 0 0"/>
       <axis xyz="0 1 0"/>
       <dynamics damping="0.2"/>
@@ -83,5 +83,5 @@
       <parent link="${prefix}base_link"/>
       <child link="${prefix}right_wheel"/>
-      <origin xyz="-${rear_wheels_axis_offset} ${rear_wheels_distance/2} ${rear_wheel_ground_offset}" rpy="0 0 0"/>
+      <origin xyz="0 ${rear_wheels_distance/2} ${rear_wheel_ground_offset}" rpy="0 0 0"/>
       <axis xyz="0 1 0"/>
       <dynamics damping="0.2"/>

Commit message: Updated wheel separation

File: ros/src/rosbot_description/urdf/rosbot.urdf.xacro (robot description, xacro)
@@ -18,5 +18,5 @@
     <xacro:property name="rear_wheel_ground_offset" value="0.0975" />
     <xacro:property name="rear_wheels_axis_offset" value="0.1" />
-    <xacro:property name="rear_wheels_distance" value="0.2476" />
+    <xacro:property name="wheel_separation" value="0.241" />
     <!-- Space btw top of beam and the each joint -->
     <!-- robot is 300mm wide, 460mm long, 170mm tall -->
@@ -55,5 +55,5 @@
       <parent link="${prefix}base_link"/>
       <child link="${prefix}left_wheel"/>
-      <origin xyz="0 -${rear_wheels_distance/2} ${rear_wheel_ground_offset}" rpy="0 0 0"/>
+      <origin xyz="0 -${wheel_separation/2} ${rear_wheel_ground_offset}" rpy="0 0 0"/>
       <axis xyz="0 1 0"/>
       <dynamics damping="0.2"/>
@@ -83,5 +83,5 @@
       <parent link="${prefix}base_link"/>
       <child link="${prefix}right_wheel"/>
-      <origin xyz="0 ${rear_wheels_distance/2} ${rear_wheel_ground_offset}" rpy="0 0 0"/>
+      <origin xyz="0 ${wheel_separation/2} ${rear_wheel_ground_offset}" rpy="0 0 0"/>
       <axis xyz="0 1 0"/>
       <dynamics damping="0.2"/>

Commit message: Restored rear wheels distance property

File: ros/src/rosbot_description/urdf/rosbot.urdf.xacro (robot description, xacro)
@@ -18,5 +18,5 @@
     <xacro:property name="rear_wheel_ground_offset" value="0.0975" />
     <xacro:property name="rear_wheels_axis_offset" value="0.1" />
-    <xacro:property name="wheel_separation" value="0.241" />
+    <xacro:property name="rear_wheels_distance" value="0.241" />
     <!-- Space btw top of beam and the each joint -->
     <!-- robot is 300mm wide, 460mm long, 170mm tall -->
@@ -55,5 +55,5 @@
       <parent link="${prefix}base_link"/>
       <child link="${prefix}left_wheel"/>
-      <origin xyz="0 -${wheel_separation/2} ${rear_wheel_ground_offset}" rpy="0 0 0"/>
+      <origin xyz="0 -${rear_wheels_distance/2} ${rear_wheel_ground_offset}" rpy="0 0 0"/>
       <axis xyz="0 1 0"/>
       <dynamics damping="0.2"/>
@@ -83,5 +83,5 @@
       <parent link="${prefix}base_link"/>
       <child link="${prefix}right_wheel"/>
-      <origin xyz="0 ${wheel_separation/2} ${rear_wheel_ground_offset}" rpy="0 0 0"/>
+      <origin xyz="0 ${rear_wheels_distance/2} ${rear_wheel_ground_offset}" rpy="0 0 0"/>
       <axis xyz="0 1 0"/>
       <dynamics damping="0.2"/>

Commit message: Added lidar link and joint

File: ros/src/rosbot_description/urdf/rosbot.urdf.xacro (robot description, xacro)
@@ -7,8 +7,10 @@
     <xacro:property name="PI" value="3.1415926535897931"/>
     <xacro:property name="base_mass" value="6.0" />
-    <!-- arbitrary value for base mass -->
     <xacro:property name="base_width" value="0.46" />
     <xacro:property name="base_length" value="0.3" />
     <xacro:property name="base_height" value="0.17" />
+    <xacro:property name="lidar_width" value="0.055" />
+    <xacro:property name="lidar_length" value="0.055" />
+    <xacro:property name="lidar_height" value="0.055" />
     <xacro:property name="wheel_mass" value="0.5" />
     <!-- arbitrary value for wheel mass -->
@@ -52,4 +54,5 @@
       </inertial>
     </link>
+    <!-- left wheel -->
     <joint name="${prefix}left_wheel_joint" type="continuous">
       <parent link="${prefix}base_link"/>
@@ -59,5 +62,4 @@
       <dynamics damping="0.2"/>
     </joint>
-    <!-- left wheel Link -->
     <link name="${prefix}left_wheel">
       <collision>
@@ -80,4 +82,5 @@
       </inertial>
     </link>
+    <!-- right wheel -->
     <joint name="${prefix}right_wheel_joint" type="continuous">
       <parent link="${prefix}base_link"/>
@@ -87,5 +90,4 @@
       <dynamics damping="0.2"/>
     </joint>
-    <!-- right wheel Link -->
     <link name="${prefix}right_wheel">
       <collision>
@@ -108,4 +110,20 @@
       </inertial>
     </link>
+    <!-- lidar -->
+    <joint name="${prefix}lidar_joint" type="continuous">
+      <parent link="${prefix}base_link"/>
+      <child link="${prefix}lidar"/>
+      <origin xyz="0 0 ${base_height + frame_ground_offset}" rpy="0 0 0"/>
+      <axis xyz="0 0 1"/>
+    </joint>
+    <link name="${prefix}lidar">
+      <visual>
+        <origin xyz="0 0 ${base_height + frame_ground_offset}" rpy="0 0 0"/>
+        <geometry>
+          <box size="${lidar_width} ${lidar_length} ${lidar_height}"/>
+        </geometry>
+        <material name="orange"/>
+      </visual>
+    </link>
   </xacro:macro>
 </robot>

Commit message: Improved robot urdf, changed lidar frame id

File: ros/src/rosbot_description/urdf/rosbot.urdf.xacro (robot description, xacro)
@@ -114,14 +114,14 @@
       <parent link="${prefix}base_link"/>
       <child link="${prefix}lidar"/>
-      <origin xyz="0 0 ${base_height + frame_ground_offset}" rpy="0 0 0"/>
+      <origin xyz="0 0 ${base_height + frame_ground_offset + lidar_height / 2}" rpy="0 0 0"/>
       <axis xyz="0 0 1"/>
     </joint>
     <link name="${prefix}lidar">
       <visual>
-        <origin xyz="0 0 ${base_height + frame_ground_offset}" rpy="0 0 0"/>
+        <origin xyz="0 0 ${base_height + frame_ground_offset + lidar_height / 2}" rpy="0 0 0"/>
         <geometry>
           <box size="${lidar_width} ${lidar_length} ${lidar_height}"/>
         </geometry>
-        <material name="orange"/>
+        <material name="green"/>
       </visual>
     </link>

Commit message: Changed lidar joint to fixed

File: ros/src/rosbot_description/urdf/rosbot.urdf.xacro (robot description, xacro)
@@ -111,6 +111,6 @@
     </link>
     <!-- lidar -->
-    <joint name="${prefix}lidar_joint" type="continuous">
-      <parent link="${prefix}base_link"/>
+    <joint name="${prefix}lidar_joint" type="fixed">
+      <parent link="${prefix}odom"/>
       <child link="${prefix}lidar"/>
       <origin xyz="0 0 ${base_height + frame_ground_offset + lidar_height / 2}" rpy="0 0 0"/>
