Commit message: Changed lidar urdf parent

File: ros/src/rosbot_description/urdf/rosbot.urdf.xacro (robot description, xacro)
@@ -7,7 +7,7 @@
     <xacro:property name="PI" value="3.1415926535897931"/>
     <xacro:property name="base_mass" value="6.0" />
-    <xacro:property name="base_width" value="0.46" />
-    <xacro:property name="base_length" value="0.3" />
-    <xacro:property name="base_height" value="0.17" />
+    <xacro:property name="body_width" value="0.46" />
+    <xacro:property name="body_length" value="0.3" />
+    <xacro:property name="body_height" value="0.17" />
     <xacro:property name="lidar_width" value="0.055" />
     <xacro:property name="lidar_length" value="0.055" />
@@ -33,25 +33,46 @@
     <!-- large wheel pulley has 72 teeth -->
     <!-- motor to wheel gear ratio is 72/16 = 4.5 -->
-    <!-- Base Link -->
+    <!-- base link -->
     <link name="${prefix}base_link">
       <collision>
-        <origin xyz="${rear_wheels_axis_offset} 0 ${base_height/2 + frame_ground_offset}" rpy="0 0 0"/>
+        <origin xyz="${rear_wheels_axis_offset} 0 ${body_height/2 + frame_ground_offset}" rpy="0 0 0"/>
         <geometry>
-          <box size="${base_width} ${base_length} ${base_height}"/>
+          <box size="${body_width} ${body_length} ${body_height}"/>
         </geometry>
       </collision>
       <visual>
-        <origin xyz="${rear_wheels_axis_offset} 0 ${base_height/2 + frame_ground_offset}" rpy="0 0 0"/>
+        <origin xyz="${rear_wheels_axis_offset} 0 ${body_height/2 + frame_ground_offset}" rpy="0 0 0"/>
         <geometry>
-          <box size="${base_width} ${base_length} ${base_height}"/>
+          <box size="${body_width} ${body_length} ${body_height}"/>
         </geometry>
         <material name="orange"/>
       </visual>
+      <!-- <inertial>
+        <origin xyz="${rear_wheels_axis_offset} 0 ${body_height/2 + frame_ground_offset}" rpy="0 0 0"/>
+        <mass value="${base_mass}"/>
+        <inertia ixx="${base_mass / 12.0 * (body_length*body_length + body_height*body_height)}" ixy="0.0" ixz="0.0" iyy="${base_mass / 12.0 * (body_height*body_height + body_width*body_width)}" iyz="0.0" izz="${base_mass / 12.0 * (body_width*body_width + body_length*body_length)}"/>
+      </inertial> -->
+    </link>
+    <!-- body -->
+    <!-- <joint name="${prefix}body_joint" type="fixed">
+      <parent link="${prefix}base_link"/>
+      <child link="${prefix}body"/>
+      <origin xyz="0 0 ${body_height + frame_ground_offset + lidar_height / 2}" rpy="0 0 0"/>
+      <axis xyz="0 0 1"/>
+    </joint>
+    <link name="${prefix}body">
+      <visual>
+        <origin xyz="0 0 ${body_height + frame_ground_offset + lidar_height / 2}" rpy="0 0 0"/>
+        <geometry>
+          <box size="${lidar_width} ${lidar_length} ${lidar_height}"/>
+        </geometry>
+        <material name="green"/>
+      </visual>
       <inertial>
-        <origin xyz="${rear_wheels_axis_offset} 0 ${base_height/2 + frame_ground_offset}" rpy="0 0 0"/>
+        <origin xyz="${rear_wheels_axis_offset} 0 ${body_height/2 + frame_ground_offset}" rpy="0 0 0"/>
         <mass value="${base_mass}"/>
-        <inertia ixx="${base_mass / 12.0 * (base_length*base_length + base_height*base_height)}" ixy="0.0" ixz="0.0" iyy="${base_mass / 12.0 * (base_height*base_height + base_width*base_width)}" iyz="0.0" izz="${base_mass / 12.0 * (base_width*base_width + base_length*base_length)}"/>
+        <inertia ixx="${base_mass / 12.0 * (body_length*body_length + body_height*body_height)}" ixy="0.0" ixz="0.0" iyy="${base_mass / 12.0 * (body_height*body_height + body_width*body_width)}" iyz="0.0" izz="${base_mass / 12.0 * (body_width*body_width + body_length*body_length)}"/>
       </inertial>
-    </link>
+    </link> -->
     <!-- left wheel -->
     <joint name="${prefix}left_wheel_joint" type="continuous">
@@ -112,12 +133,12 @@
     <!-- lidar -->
     <joint name="${prefix}lidar_joint" type="fixed">
-      <parent link="${prefix}odom"/>
+      <parent link="${prefix}base_link"/>
       <child link="${prefix}lidar"/>
-      <origin xyz="0 0 ${base_height + frame_ground_offset + lidar_height / 2}" rpy="0 0 0"/>
+      <origin xyz="0 0 ${body_height + frame_ground_offset + lidar_height / 2}" rpy="0 0 0"/>
       <axis xyz="0 0 1"/>
     </joint>
     <link name="${prefix}lidar">
       <visual>
-        <origin xyz="0 0 ${base_height + frame_ground_offset + lidar_height / 2}" rpy="0 0 0"/>
+        <origin xyz="0 0 ${body_height + frame_ground_offset + lidar_height / 2}" rpy="0 0 0"/>
         <geometry>
           <box size="${lidar_width} ${lidar_length} ${lidar_height}"/>

Commit message: Updated lidar urdf

File: ros/src/rosbot_description/urdf/rosbot.urdf.xacro (robot description, xacro)
@@ -135,10 +135,10 @@
       <parent link="${prefix}base_link"/>
       <child link="${prefix}lidar"/>
-      <origin xyz="0 0 ${body_height + frame_ground_offset + lidar_height / 2}" rpy="0 0 0"/>
+      <origin xyz="0 0 ${body_height/2 + lidar_height/2}" rpy="0 0 0"/>
       <axis xyz="0 0 1"/>
     </joint>
     <link name="${prefix}lidar">
       <visual>
-        <origin xyz="0 0 ${body_height + frame_ground_offset + lidar_height / 2}" rpy="0 0 0"/>
+        <origin xyz="0 0 0" rpy="0 0 0"/>
         <geometry>
           <box size="${lidar_width} ${lidar_length} ${lidar_height}"/>

File: ros/src/rosbot_description/urdf/rosbot_system.urdf.xacro (robot description, xacro)
@@ -11,4 +11,4 @@
   <xacro:rosbot prefix="$(arg prefix)" />
   <xacro:rosbot_gazebo prefix="$(arg prefix)" />
-  <xacro:rosbot_system name="DiffBotSystem" prefix="$(arg prefix)" use_fake_hardware="$(arg use_fake_hardware)" fake_sensor_commands="$(arg fake_sensor_commands)"/>
+  <xacro:rosbot_system name="RosbotSystem" prefix="$(arg prefix)" use_fake_hardware="$(arg use_fake_hardware)" fake_sensor_commands="$(arg fake_sensor_commands)"/>
 </robot>

Commit message: Updated lidar link origin

File: ros/src/rosbot_description/urdf/rosbot.urdf.xacro (robot description, xacro)
@@ -140,5 +140,5 @@
     <link name="${prefix}lidar">
       <visual>
-        <origin xyz="0 0 0" rpy="0 0 0"/>
+        <origin xyz="0 0 ${body_height/2 + lidar_height/2}" rpy="0 0 0"/>
         <geometry>
           <box size="${lidar_width} ${lidar_length} ${lidar_height}"/>

Commit message: Working on lidar transform

File: ros/src/rosbot_description/urdf/rosbot.urdf.xacro (robot description, xacro)
@@ -135,10 +135,10 @@
       <parent link="${prefix}base_link"/>
       <child link="${prefix}lidar"/>
-      <origin xyz="${-rear_wheels_axis_offset} 0 ${body_height/2 + lidar_height/2}" rpy="0 0 0"/>
+      <origin xyz="${rear_wheels_axis_offset} 0 ${frame_ground_offset + body_height/2 + lidar_height}" rpy="0 0 0"/>
       <axis xyz="0 0 1"/>
     </joint>
     <link name="${prefix}lidar">
       <visual>
-        <origin xyz="${-rear_wheels_axis_offset} 0 ${body_height/2 + lidar_height/2}" rpy="0 0 0"/>
+        <origin xyz="0 0 0" rpy="0 0 0"/>
         <geometry>
           <box size="${lidar_width} ${lidar_length} ${lidar_height}"/>

Commit message: Improved lidar joint origin

File: ros/src/rosbot_description/urdf/rosbot.urdf.xacro (robot description, xacro)
@@ -135,5 +135,5 @@
       <parent link="${prefix}base_link"/>
       <child link="${prefix}lidar"/>
-      <origin xyz="${rear_wheels_axis_offset} 0 ${frame_ground_offset + body_height/2 + lidar_height}" rpy="0 0 0"/>
+      <origin xyz="${rear_wheels_axis_offset} 0 ${frame_ground_offset + body_height + lidar_height / 2}" rpy="0 0 0"/>
       <axis xyz="0 0 1"/>
     </joint>

Commit message: Rotated lidar origin 180 degrees

File: ros/src/rosbot_description/urdf/rosbot.urdf.xacro (robot description, xacro)
@@ -140,5 +140,5 @@
     <link name="${prefix}lidar">
       <visual>
-        <origin xyz="0 0 0" rpy="0 0 0"/>
+        <origin xyz="0 0 0" rpy="0 0 ${PI/2}"/>
         <geometry>
           <box size="${lidar_width} ${lidar_length} ${lidar_height}"/>

Commit message: Fixed lidar joint origin rotation

File: ros/src/rosbot_description/urdf/rosbot.urdf.xacro (robot description, xacro)
@@ -135,10 +135,10 @@
       <parent link="${prefix}base_link"/>
       <child link="${prefix}lidar"/>
-      <origin xyz="${rear_wheels_axis_offset} 0 ${frame_ground_offset + body_height + lidar_height / 2}" rpy="0 0 0"/>
+      <origin xyz="${rear_wheels_axis_offset} 0 ${frame_ground_offset + body_height + lidar_height / 2}" rpy="0 0 ${PI}"/>
       <axis xyz="0 0 1"/>
     </joint>
     <link name="${prefix}lidar">
       <visual>
-        <origin xyz="0 0 0" rpy="0 0 ${PI/2}"/>
+        <origin xyz="0 0 0" rpy="0 0 0"/>
         <geometry>
           <box size="${lidar_width} ${lidar_length} ${lidar_height}"/>

Commit message: Improved robot description, added test body mesh, made lidar cylinder

File: ros/src/rosbot_description/urdf/rosbot.urdf.xacro (robot description, xacro)
@@ -4,22 +4,24 @@
 <robot xmlns:xacro="http://www.ros.org/wiki/xacro">
   <xacro:macro name="rosbot" params="prefix">
-    <!-- Constants for robot dimensions -->
+    <!-- constants -->
     <xacro:property name="PI" value="3.1415926535897931"/>
-    <xacro:property name="base_mass" value="6.0" />
+    <!-- body properties -->
+    <xacro:property name="body_mass" value="6.0" />
     <xacro:property name="body_width" value="0.46" />
     <xacro:property name="body_length" value="0.3" />
     <xacro:property name="body_height" value="0.17" />
-    <xacro:property name="lidar_width" value="0.055" />
-    <xacro:property name="lidar_length" value="0.055" />
+    <xacro:property name="body_ground_offset" value="0.0575" />
+    <!-- lidar properties -->
+    <!-- <xacro:property name="lidar_width" value="0.055" /> -->
+    <!-- <xacro:property name="lidar_length" value="0.055" /> -->
     <xacro:property name="lidar_height" value="0.055" />
-    <xacro:property name="wheel_mass" value="0.5" />
-    <!-- arbitrary value for wheel mass -->
-    <xacro:property name="wheel_len" value="0.05" />
-    <xacro:property name="wheel_radius" value="0.0975" />
-    <xacro:property name="frame_ground_offset" value="0.0575" />
+    <xacro:property name="lidar_radius" value="0.0275" />
+    <!-- rear wheel properties -->
+    <xacro:property name="real_wheel_mass" value="0.5" />
+    <xacro:property name="rear_wheel_width" value="0.05" />
+    <xacro:property name="rear_wheel_radius" value="0.0975" />
     <xacro:property name="rear_wheel_ground_offset" value="0.0975" />
-    <xacro:property name="rear_wheels_axis_offset" value="0.1" />
-    <xacro:property name="rear_wheels_distance" value="0.241" />
-    <!-- Space btw top of beam and the each joint -->
+    <xacro:property name="rear_wheel_axis_offset" value="0.1" />
+    <xacro:property name="rear_wheel_distance" value="0.241" />
     <!-- robot is 300mm wide, 460mm long, 170mm tall -->
     <!-- front wheels are 38.5mm off the ground surface -->
@@ -36,5 +38,5 @@
     <link name="${prefix}base_link">
       <collision>
-        <origin xyz="${rear_wheels_axis_offset} 0 ${body_height/2 + frame_ground_offset}" rpy="0 0 0"/>
+        <origin xyz="${rear_wheel_axis_offset} 0 ${body_height/2 + body_ground_offset}" rpy="0 0 0"/>
         <geometry>
           <box size="${body_width} ${body_length} ${body_height}"/>
@@ -42,14 +44,16 @@
       </collision>
       <visual>
-        <origin xyz="${rear_wheels_axis_offset} 0 ${body_height/2 + frame_ground_offset}" rpy="0 0 0"/>
+        <origin xyz="${rear_wheel_axis_offset} 0 ${body_height/2 + body_ground_offset}" rpy="0 0 0"/>
         <geometry>
-          <box size="${body_width} ${body_length} ${body_height}"/>
+          <!-- <box size="${body_width} ${body_length} ${body_height}"/> -->
+          <!-- TODO: replace simple box with robot mesh -->
+          <mesh filename="package://rosbot_description/meshes/rosbot_body.stl" scale="0.001 0.001 0.001"/>
         </geometry>
         <material name="orange"/>
       </visual>
       <!-- <inertial>
-        <origin xyz="${rear_wheels_axis_offset} 0 ${body_height/2 + frame_ground_offset}" rpy="0 0 0"/>
-        <mass value="${base_mass}"/>
-        <inertia ixx="${base_mass / 12.0 * (body_length*body_length + body_height*body_height)}" ixy="0.0" ixz="0.0" iyy="${base_mass / 12.0 * (body_height*body_height + body_width*body_width)}" iyz="0.0" izz="${base_mass / 12.0 * (body_width*body_width + body_length*body_length)}"/>
+        <origin xyz="${rear_wheel_axis_offset} 0 ${body_height/2 + body_ground_offset}" rpy="0 0 0"/>
+        <mass value="${body_mass}"/>
+        <inertia ixx="${body_mass / 12.0 * (body_length*body_length + body_height*body_height)}" ixy="0.0" ixz="0.0" iyy="${body_mass / 12.0 * (body_height*body_height + body_width*body_width)}" iyz="0.0" izz="${body_mass / 12.0 * (body_width*body_width + body_length*body_length)}"/>
       </inertial> -->
     </link>
@@ -58,10 +62,10 @@
       <parent link="${prefix}base_link"/>
       <child link="${prefix}body"/>
-      <origin xyz="0 0 ${body_height + frame_ground_offset + lidar_height / 2}" rpy="0 0 0"/>
+      <origin xyz="0 0 ${body_height + body_ground_offset + lidar_height / 2}" rpy="0 0 0"/>
       <axis xyz="0 0 1"/>
     </joint>
     <link name="${prefix}body">
       <visual>
-        <origin xyz="0 0 ${body_height + frame_ground_offset + lidar_height / 2}" rpy="0 0 0"/>
+        <origin xyz="0 0 ${body_height + body_ground_offset + lidar_height / 2}" rpy="0 0 0"/>
         <geometry>
           <box size="${lidar_width} ${lidar_length} ${lidar_height}"/>
@@ -70,7 +74,7 @@
       </visual>
       <inertial>
-        <origin xyz="${rear_wheels_axis_offset} 0 ${body_height/2 + frame_ground_offset}" rpy="0 0 0"/>
-        <mass value="${base_mass}"/>
-        <inertia ixx="${base_mass / 12.0 * (body_length*body_length + body_height*body_height)}" ixy="0.0" ixz="0.0" iyy="${base_mass / 12.0 * (body_height*body_height + body_width*body_width)}" iyz="0.0" izz="${base_mass / 12.0 * (body_width*body_width + body_length*body_length)}"/>
+        <origin xyz="${rear_wheel_axis_offset} 0 ${body_height/2 + body_ground_offset}" rpy="0 0 0"/>
+        <mass value="${body_mass}"/>
+        <inertia ixx="${body_mass / 12.0 * (body_length*body_length + body_height*body_height)}" ixy="0.0" ixz="0.0" iyy="${body_mass / 12.0 * (body_height*body_height + body_width*body_width)}" iyz="0.0" izz="${body_mass / 12.0 * (body_width*body_width + body_length*body_length)}"/>
       </inertial>
     </link> -->
@@ -79,5 +83,5 @@
       <parent link="${prefix}base_link"/>
       <child link="${prefix}left_wheel"/>
-      <origin xyz="0 -${rear_wheels_distance/2} ${rear_wheel_ground_offset}" rpy="0 0 0"/>
+      <origin xyz="0 -${rear_wheel_distance/2} ${rear_wheel_ground_offset}" rpy="0 0 0"/>
       <axis xyz="0 1 0"/>
       <dynamics damping="0.2"/>
@@ -87,5 +91,5 @@
         <origin xyz="0 0 0" rpy="${PI/2} 0 0"/>
         <geometry>
-          <cylinder length="${wheel_len}" radius="${wheel_radius}"/>
+          <cylinder length="${rear_wheel_width}" radius="${rear_wheel_radius}"/>
         </geometry>
       </collision>
@@ -93,5 +97,5 @@
         <origin xyz="0 0 0" rpy="${PI/2} 0 0"/>
         <geometry>
-          <cylinder length="${wheel_len}" radius="${wheel_radius}"/>
+          <cylinder length="${rear_wheel_width}" radius="${rear_wheel_radius}"/>
         </geometry>
         <material name="black"/>
@@ -99,6 +103,6 @@
       <inertial>
         <origin xyz="0 0 0" rpy="${PI/2} 0 0"/>
-        <mass value="${wheel_mass}"/>
-        <inertia ixx="${wheel_mass / 12.0 * (3*wheel_radius + wheel_len*wheel_len)}" ixy="0.0" ixz="0.0" iyy="${wheel_mass / 12.0 * wheel_radius*wheel_radius}" iyz="0.0" izz="${wheel_mass / 12.0 * wheel_radius*wheel_radius}"/>
+        <mass value="${real_wheel_mass}"/>
+        <inertia ixx="${real_wheel_mass / 12.0 * (3*rear_wheel_radius + rear_wheel_width*rear_wheel_width)}" ixy="0.0" ixz="0.0" iyy="${real_wheel_mass / 12.0 * rear_wheel_radius*rear_wheel_radius}" iyz="0.0" izz="${real_wheel_mass / 12.0 * rear_wheel_radius*rear_wheel_radius}"/>
       </inertial>
     </link>
@@ -107,5 +111,5 @@
       <parent link="${prefix}base_link"/>
       <child link="${prefix}right_wheel"/>
-      <origin xyz="0 ${rear_wheels_distance/2} ${rear_wheel_ground_offset}" rpy="0 0 0"/>
+      <origin xyz="0 ${rear_wheel_distance/2} ${rear_wheel_ground_offset}" rpy="0 0 0"/>
       <axis xyz="0 1 0"/>
       <dynamics damping="0.2"/>
@@ -115,5 +119,5 @@
         <origin xyz="0 0 0" rpy="${PI/2} 0 0"/>
         <geometry>
-          <cylinder length="${wheel_len}" radius="${wheel_radius}"/>
+          <cylinder length="${rear_wheel_width}" radius="${rear_wheel_radius}"/>
         </geometry>
       </collision>
@@ -121,5 +125,5 @@
         <origin xyz="0 0 0" rpy="${PI/2} 0 0"/>
         <geometry>
-          <cylinder length="${wheel_len}" radius="${wheel_radius}"/>
+          <cylinder length="${rear_wheel_width}" radius="${rear_wheel_radius}"/>
         </geometry>
         <material name="black"/>
@@ -127,6 +131,6 @@
       <inertial>
         <origin xyz="0 0 0" rpy="${PI/2} 0 0"/>
-        <mass value="${wheel_mass}"/>
-        <inertia ixx="${wheel_mass / 12.0 * (3*wheel_radius + wheel_len*wheel_len)}" ixy="0.0" ixz="0.0" iyy="${wheel_mass / 12.0 * wheel_radius*wheel_radius}" iyz="0.0" izz="${wheel_mass / 12.0 * wheel_radius*wheel_radius}"/>
+        <mass value="${real_wheel_mass}"/>
+        <inertia ixx="${real_wheel_mass / 12.0 * (3*rear_wheel_radius + rear_wheel_width*rear_wheel_width)}" ixy="0.0" ixz="0.0" iyy="${real_wheel_mass / 12.0 * rear_wheel_radius*rear_wheel_radius}" iyz="0.0" izz="${real_wheel_mass / 12.0 * rear_wheel_radius*rear_wheel_radius}"/>
       </inertial>
     </link>
@@ -135,5 +139,5 @@
       <parent link="${prefix}base_link"/>
       <child link="${prefix}lidar"/>
-      <origin xyz="${rear_wheels_axis_offset} 0 ${frame_ground_offset + body_height + lidar_height / 2}" rpy="0 0 ${PI}"/>
+      <origin xyz="${rear_wheel_axis_offset} 0 ${body_ground_offset + body_height + lidar_height / 2}" rpy="0 0 ${PI}"/>
       <axis xyz="0 0 1"/>
     </joint>
@@ -142,5 +146,6 @@
         <origin xyz="0 0 0" rpy="0 0 0"/>
         <geometry>
-          <box size="${lidar_width} ${lidar_length} ${lidar_height}"/>
+          <!-- <box size="${lidar_width} ${lidar_length} ${lidar_height}"/> -->
+          <cylinder length="${lidar_height}" radius="${lidar_radius}"/>
         </geometry>
         <material name="green"/>

Commit message: Testing mesh scale

File: ros/src/rosbot_description/urdf/rosbot.urdf.xacro (robot description, xacro)
@@ -48,5 +48,5 @@
           <!-- <box size="${body_width} ${body_length} ${body_height}"/> -->
           <!-- TODO replace simple box with robot mesh -->
-          <mesh filename="package://rosbot_description/meshes/rosbot_body.stl" scale="0.001 0.001 0.001"/>
+          <mesh filename="package://rosbot_description/meshes/rosbot_body.stl" scale="1 1 1"/>
         </geometry>
         <material name="orange"/>

Commit message: Restored simple box body visualization

File: ros/src/rosbot_description/urdf/rosbot.urdf.xacro (robot description, xacro)
@@ -46,7 +46,7 @@
         <origin xyz="${rear_wheel_axis_offset} 0 ${body_height/2 + body_ground_offset}" rpy="0 0 0"/>
         <geometry>
-          <!-- <box size="${body_width} ${body_length} ${body_height}"/> -->
+          <box size="${body_width} ${body_length} ${body_height}"/>
           <!-- TODO replace simple box with robot mesh -->
-          <mesh filename="package://rosbot_description/meshes/rosbot_body.stl" scale="1 1 1"/>
+          <!-- <mesh filename="package://rosbot_description/meshes/rosbot_body.stl" scale="0.001 0.001 0.001"/> -->
         </geometry>
         <material name="orange"/>

Commit message: Renamed lidar link to base_laser

File: ros/src/rosbot_description/urdf/rosbot.urdf.xacro (robot description, xacro)
@@ -138,9 +138,9 @@
     <joint name="${prefix}lidar_joint" type="fixed">
       <parent link="${prefix}base_link"/>
-      <child link="${prefix}lidar"/>
+      <child link="${prefix}base_laser"/>
       <origin xyz="${rear_wheel_axis_offset} 0 ${body_ground_offset + body_height + lidar_height / 2}" rpy="0 0 ${PI}"/>
       <axis xyz="0 0 1"/>
     </joint>
-    <link name="${prefix}lidar">
+    <link name="${prefix}base_laser">
       <visual>
         <origin xyz="0 0 0" rpy="0 0 0"/>

Commit message: Removed unneeded controller manager definition

File: ros/src/rosbot_description/urdf/rosbot.urdf.xacro (robot description, xacro)
@@ -13,6 +13,4 @@
     <xacro:property name="body_ground_offset" value="0.0575" />
     <!-- lidar properties -->
-    <!-- <xacro:property name="lidar_width" value="0.055" /> -->
-    <!-- <xacro:property name="lidar_length" value="0.055" /> -->
     <xacro:property name="lidar_height" value="0.055" />
     <xacro:property name="lidar_radius" value="0.0275" />
@@ -24,4 +22,5 @@
     <xacro:property name="rear_wheel_axis_offset" value="0.1" />
     <xacro:property name="rear_wheel_distance" value="0.241" />
+    <!-- PHYSICAL ROBOT MEASUREMENTS -->
     <!-- robot is 300mm wide, 460mm long, 170mm tall -->
     <!-- front wheels are 38.5mm off the ground surface -->

Commit message: Added base footprint

File: ros/src/rosbot_description/urdf/rosbot.urdf.xacro (robot description, xacro)
@@ -34,8 +34,15 @@
     <!-- large wheel pulley has 72 teeth -->
     <!-- motor to wheel gear ratio is 72/16 = 4.5 -->
+    <!-- base footprint -->
+    <link name="base_footprint"/>
     <!-- base link -->
+    <joint name="base_joint" type="fixed">
+      <parent link="base_footprint"/>
+      <child link="base_link" />
+      <origin xyz="0 0 ${body_ground_offset + body_height/2}" rpy="0 0 0"/>
+    </joint>
     <link name="${prefix}base_link">
       <collision>
-        <origin xyz="${rear_wheel_axis_offset} 0 ${body_height/2 + body_ground_offset}" rpy="0 0 0"/>
+        <origin xyz="${rear_wheel_axis_offset} 0 0" rpy="0 0 0"/>
         <geometry>
           <box size="${body_width} ${body_length} ${body_height}"/>
@@ -43,5 +50,5 @@
       </collision>
       <visual>
-        <origin xyz="${rear_wheel_axis_offset} 0 ${body_height/2 + body_ground_offset}" rpy="0 0 0"/>
+        <origin xyz="${rear_wheel_axis_offset} 0 0" rpy="0 0 0"/>
         <geometry>
           <box size="${body_width} ${body_length} ${body_height}"/>
@@ -52,5 +59,5 @@
       </visual>
       <!-- <inertial>
-        <origin xyz="${rear_wheel_axis_offset} 0 ${body_height/2 + body_ground_offset}" rpy="0 0 0"/>
+        <origin xyz="${rear_wheel_axis_offset} 0 0" rpy="0 0 0"/>
         <mass value="${body_mass}"/>
         <inertia ixx="${body_mass / 12.0 * (body_length*body_length + body_height*body_height)}" ixy="0.0" ixz="0.0" iyy="${body_mass / 12.0 * (body_height*body_height + body_width*body_width)}" iyz="0.0" izz="${body_mass / 12.0 * (body_width*body_width + body_length*body_length)}"/>
