Commit message: Working on base footprint urdf

File: ros/src/rosbot_description/urdf/rosbot.urdf.xacro (robot description, xacro)
@@ -37,7 +37,7 @@
     <link name="base_footprint"/>
     <!-- base link -->
-    <joint name="base_joint" type="fixed">
-      <parent link="base_footprint"/>
-      <child link="base_link" />
+    <joint name="${prefix}base_joint" type="fixed">
+      <parent link="${prefix}base_footprint"/>
+      <child link="${prefix}base_link" />
       <origin xyz="0 0 ${body_ground_offset + body_height/2}" rpy="0 0 0"/>
     </joint>

Commit message: Improved robot description

File: ros/src/rosbot_description/urdf/rosbot.urdf.xacro (robot description, xacro)
@@ -40,9 +40,9 @@
       <parent link="${prefix}base_footprint"/>
       <child link="${prefix}base_link" />
-      <origin xyz="0 0 ${body_ground_offset + body_height/2}" rpy="0 0 0"/>
+      <origin xyz="0 0 ${body_ground_offset}" rpy="0 0 0"/>
     </joint>
     <link name="${prefix}base_link">
       <collision>
-        <origin xyz="${rear_wheel_axis_offset} 0 0" rpy="0 0 0"/>
+        <origin xyz="${rear_wheel_axis_offset} 0 ${body_height/2}" rpy="0 0 0"/>
         <geometry>
           <box size="${body_width} ${body_length} ${body_height}"/>
@@ -50,5 +50,5 @@
       </collision>
       <visual>
-        <origin xyz="${rear_wheel_axis_offset} 0 0" rpy="0 0 0"/>
+        <origin xyz="${rear_wheel_axis_offset} 0 0" rpy="0 0 body_height/2"/>
         <geometry>
           <box size="${body_width} ${body_length} ${body_height}"/>
@@ -89,5 +89,5 @@
       <parent link="${prefix}base_link"/>
       <child link="${prefix}left_wheel"/>
-      <origin xyz="0 -${rear_wheel_distance/2} ${rear_wheel_ground_offset}" rpy="0 0 0"/>
+      <origin xyz="0 -${rear_wheel_distance/2} 0" rpy="0 0 0"/>
       <axis xyz="0 1 0"/>
       <dynamics damping="0.2"/>
@@ -117,5 +117,5 @@
       <parent link="${prefix}base_link"/>
       <child link="${prefix}right_wheel"/>
-      <origin xyz="0 ${rear_wheel_distance/2} ${rear_wheel_ground_offset}" rpy="0 0 0"/>
+      <origin xyz="0 ${rear_wheel_distance/2} 0" rpy="0 0 0"/>
       <axis xyz="0 1 0"/>
       <dynamics damping="0.2"/>

Commit message: Improved robot description

File: ros/src/rosbot_description/urdf/rosbot.urdf.xacro (robot description, xacro)
@@ -50,5 +50,5 @@
       </collision>
       <visual>
-        <origin xyz="${rear_wheel_axis_offset} 0 0" rpy="0 0 body_height/2"/>
+        <origin xyz="${rear_wheel_axis_offset} 0 0" rpy="0 0 ${body_height/2}"/>
         <geometry>
           <box size="${body_width} ${body_length} ${body_height}"/>

Commit message: Working on link offsets

File: ros/src/rosbot_description/urdf/rosbot.urdf.xacro (robot description, xacro)
@@ -40,9 +40,9 @@
       <parent link="${prefix}base_footprint"/>
       <child link="${prefix}base_link" />
-      <origin xyz="0 0 ${body_ground_offset}" rpy="0 0 0"/>
+      <origin xyz="0 0 ${rear_wheel_ground_offset}" rpy="0 0 0"/>
     </joint>
     <link name="${prefix}base_link">
       <collision>
-        <origin xyz="${rear_wheel_axis_offset} 0 ${body_height/2}" rpy="0 0 0"/>
+        <origin xyz="${rear_wheel_axis_offset} 0 ${(rear_wheel_ground_offset - body_ground_offset) + body_height/2}" rpy="0 0 0"/>
         <geometry>
           <box size="${body_width} ${body_length} ${body_height}"/>
@@ -50,5 +50,5 @@
       </collision>
       <visual>
-        <origin xyz="${rear_wheel_axis_offset} 0 0" rpy="0 0 ${body_height/2}"/>
+        <origin xyz="${rear_wheel_axis_offset} 0 0" rpy="0 0 ${(rear_wheel_ground_offset - body_ground_offset) + body_height/2}"/>
         <geometry>
           <box size="${body_width} ${body_length} ${body_height}"/>

Commit message: Working on base link offset

File: ros/src/rosbot_description/urdf/rosbot.urdf.xacro (robot description, xacro)
@@ -44,5 +44,5 @@
     <link name="${prefix}base_link">
       <collision>
-        <origin xyz="${rear_wheel_axis_offset} 0 ${(rear_wheel_ground_offset - body_ground_offset) + body_height/2}" rpy="0 0 0"/>
+        <origin xyz="${rear_wheel_axis_offset} 0 ${body_height/2 - (rear_wheel_ground_offset - body_ground_offset)}" rpy="0 0 0"/>
         <geometry>
           <box size="${body_width} ${body_length} ${body_height}"/>
@@ -50,5 +50,5 @@
       </collision>
       <visual>
-        <origin xyz="${rear_wheel_axis_offset} 0 0" rpy="0 0 ${(rear_wheel_ground_offset - body_ground_offset) + body_height/2}"/>
+        <origin xyz="${rear_wheel_axis_offset} 0 0" rpy="0 0 ${body_height/2 - (rear_wheel_ground_offset - body_ground_offset)}"/>
         <geometry>
           <box size="${body_width} ${body_length} ${body_height}"/>
@@ -145,5 +145,5 @@
       <parent link="${prefix}base_link"/>
       <child link="${prefix}base_laser"/>
-      <origin xyz="${rear_wheel_axis_offset} 0 ${body_ground_offset + body_height + lidar_height / 2}" rpy="0 0 ${PI}"/>
+      <origin xyz="${rear_wheel_axis_offset} 0 ${body_height / 2 + lidar_height / 2}" rpy="0 0 ${PI}"/>
       <axis xyz="0 0 1"/>
     </joint>

Commit message: Working on base link

File: ros/src/rosbot_description/urdf/rosbot.urdf.xacro (robot description, xacro)
@@ -50,5 +50,5 @@
       </collision>
       <visual>
-        <origin xyz="${rear_wheel_axis_offset} 0 0" rpy="0 0 ${body_height/2 - (rear_wheel_ground_offset - body_ground_offset)}"/>
+        <origin xyz="${rear_wheel_axis_offset} 0 ${body_height/2 - (rear_wheel_ground_offset - body_ground_offset)}" rpy="0 0 0"/>
         <geometry>
           <box size="${body_width} ${body_length} ${body_height}"/>

Commit message: Working on offsets

File: ros/src/rosbot_description/urdf/rosbot.urdf.xacro (robot description, xacro)
@@ -40,9 +40,9 @@
       <parent link="${prefix}base_footprint"/>
       <child link="${prefix}base_link" />
-      <origin xyz="0 0 ${rear_wheel_ground_offset}" rpy="0 0 0"/>
+      <origin xyz="0 0 ${body_ground_offset}" rpy="0 0 0"/>
     </joint>
     <link name="${prefix}base_link">
       <collision>
-        <origin xyz="${rear_wheel_axis_offset} 0 ${body_height/2 - (rear_wheel_ground_offset - body_ground_offset)}" rpy="0 0 0"/>
+        <origin xyz="${rear_wheel_axis_offset} 0 ${body_height/2}" rpy="0 0 0"/>
         <geometry>
           <box size="${body_width} ${body_length} ${body_height}"/>
@@ -50,5 +50,5 @@
       </collision>
       <visual>
-        <origin xyz="${rear_wheel_axis_offset} 0 ${body_height/2 - (rear_wheel_ground_offset - body_ground_offset)}" rpy="0 0 0"/>
+        <origin xyz="${rear_wheel_axis_offset} 0 ${body_height/2}" rpy="0 0 0"/>
         <geometry>
           <box size="${body_width} ${body_length} ${body_height}"/>
@@ -89,5 +89,5 @@
       <parent link="${prefix}base_link"/>
       <child link="${prefix}left_wheel"/>
-      <origin xyz="0 -${rear_wheel_distance/2} 0" rpy="0 0 0"/>
+      <origin xyz="0 -${rear_wheel_distance/2} (rear_wheel_ground_offset - body_ground_offset)" rpy="0 0 0"/>
       <axis xyz="0 1 0"/>
       <dynamics damping="0.2"/>
@@ -117,5 +117,5 @@
       <parent link="${prefix}base_link"/>
       <child link="${prefix}right_wheel"/>
-      <origin xyz="0 ${rear_wheel_distance/2} 0" rpy="0 0 0"/>
+      <origin xyz="0 ${rear_wheel_distance/2} (rear_wheel_ground_offset - body_ground_offset)" rpy="0 0 0"/>
       <axis xyz="0 1 0"/>
       <dynamics damping="0.2"/>

Commit message: Working on offsets

File: ros/src/rosbot_description/urdf/rosbot.urdf.xacro (robot description, xacro)
@@ -89,5 +89,5 @@
       <parent link="${prefix}base_link"/>
       <child link="${prefix}left_wheel"/>
-      <origin xyz="0 -${rear_wheel_distance/2} (rear_wheel_ground_offset - body_ground_offset)" rpy="0 0 0"/>
+      <origin xyz="0 -${rear_wheel_distance/2} ${rear_wheel_ground_offset - body_ground_offset}" rpy="0 0 0"/>
       <axis xyz="0 1 0"/>
       <dynamics damping="0.2"/>
@@ -117,5 +117,5 @@
       <parent link="${prefix}base_link"/>
       <child link="${prefix}right_wheel"/>
-      <origin xyz="0 ${rear_wheel_distance/2} (rear_wheel_ground_offset - body_ground_offset)" rpy="0 0 0"/>
+      <origin xyz="0 ${rear_wheel_distance/2} ${rear_wheel_ground_offset - body_ground_offset}" rpy="0 0 0"/>
       <axis xyz="0 1 0"/>
       <dynamics damping="0.2"/>

Commit message: Updated lidar urdf origin

File: ros/src/rosbot_description/urdf/rosbot.urdf.xacro (robot description, xacro)
@@ -145,5 +145,5 @@
       <parent link="${prefix}base_link"/>
       <child link="${prefix}base_laser"/>
-      <origin xyz="${rear_wheel_axis_offset} 0 ${body_height / 2 + lidar_height / 2}" rpy="0 0 ${PI}"/>
+      <origin xyz="${rear_wheel_axis_offset} 0 ${body_height + lidar_height / 2}" rpy="0 0 ${PI}"/>
       <axis xyz="0 0 1"/>
     </joint>

Commit message: Testing footprint origin

File: ros/src/rosbot_description/urdf/rosbot.urdf.xacro (robot description, xacro)
@@ -40,9 +40,9 @@
       <parent link="${prefix}base_footprint"/>
       <child link="${prefix}base_link" />
-      <origin xyz="0 0 ${body_ground_offset}" rpy="0 0 0"/>
+      <origin xyz="${rear_wheel_axis_offset} 0 ${body_ground_offset}" rpy="0 0 0"/>
     </joint>
     <link name="${prefix}base_link">
       <collision>
-        <origin xyz="${rear_wheel_axis_offset} 0 ${body_height/2}" rpy="0 0 0"/>
+        <origin xyz="0 0 ${body_height/2}" rpy="0 0 0"/>
         <geometry>
           <box size="${body_width} ${body_length} ${body_height}"/>
@@ -50,5 +50,5 @@
       </collision>
       <visual>
-        <origin xyz="${rear_wheel_axis_offset} 0 ${body_height/2}" rpy="0 0 0"/>
+        <origin xyz="0 0 ${body_height/2}" rpy="0 0 0"/>
         <geometry>
           <box size="${body_width} ${body_length} ${body_height}"/>

Commit message: Testing base footprint

File: ros/src/rosbot_description/urdf/rosbot.urdf.xacro (robot description, xacro)
@@ -40,9 +40,9 @@
       <parent link="${prefix}base_footprint"/>
       <child link="${prefix}base_link" />
-      <origin xyz="${rear_wheel_axis_offset} 0 ${body_ground_offset}" rpy="0 0 0"/>
+      <origin xyz="${-rear_wheel_axis_offset} 0 ${body_ground_offset}" rpy="0 0 0"/>
     </joint>
     <link name="${prefix}base_link">
       <collision>
-        <origin xyz="0 0 ${body_height/2}" rpy="0 0 0"/>
+        <origin xyz="${rear_wheel_axis_offset} 0 ${body_height/2}" rpy="0 0 0"/>
         <geometry>
           <box size="${body_width} ${body_length} ${body_height}"/>
@@ -50,5 +50,5 @@
       </collision>
       <visual>
-        <origin xyz="0 0 ${body_height/2}" rpy="0 0 0"/>
+        <origin xyz="${rear_wheel_axis_offset} 0 ${body_height/2}" rpy="0 0 0"/>
         <geometry>
           <box size="${body_width} ${body_length} ${body_height}"/>

Commit message: Restored base footprint origin

File: ros/src/rosbot_description/urdf/rosbot.urdf.xacro (robot description, xacro)
@@ -40,5 +40,5 @@
       <parent link="${prefix}base_footprint"/>
       <child link="${prefix}base_link" />
-      <origin xyz="${-rear_wheel_axis_offset} 0 ${body_ground_offset}" rpy="0 0 0"/>
+      <origin xyz="0 0 ${body_ground_offset}" rpy="0 0 0"/>
     </joint>
     <link name="${prefix}base_link">

Commit message: Added robot body urdf inertia, inertia macros

File: ros/src/rosbot_description/urdf/rosbot.urdf.xacro (robot description, xacro)
@@ -3,4 +3,6 @@
 <!-- <robot xmlns:xacro="http://www.ros.org/wiki/xacro" name="rosbot"> -->
 <robot xmlns:xacro="http://www.ros.org/wiki/xacro">
+  <!-- include inertia calculation macros -->
+  <xacro:include filename="$(find rosbot_description)/urdf/inertia.urdf.xacro" />
   <xacro:macro name="rosbot" params="prefix">
     <!-- constants -->
@@ -58,9 +60,5 @@
         <material name="orange"/>
       </visual>
-      <!-- <inertial>
-        <origin xyz="${rear_wheel_axis_offset} 0 0" rpy="0 0 0"/>
-        <mass value="${body_mass}"/>
-        <inertia ixx="${body_mass / 12.0 * (body_length*body_length + body_height*body_height)}" ixy="0.0" ixz="0.0" iyy="${body_mass / 12.0 * (body_height*body_height + body_width*body_width)}" iyz="0.0" izz="${body_mass / 12.0 * (body_width*body_width + body_length*body_length)}"/>
-      </inertial> -->
+      <xacro:box_inertia m="${body_mass}" w="${body_width}" d="${body_length}" h="${body_height}"/>
     </link>
     <!-- body -->

Commit message: Added urdf wheel inertias

File: ros/src/rosbot_description/urdf/rosbot.urdf.xacro (robot description, xacro)
@@ -105,9 +105,5 @@
         <material name="black"/>
       </visual>
-      <inertial>
-        <origin xyz="0 0 0" rpy="${PI/2} 0 0"/>
-        <mass value="${real_wheel_mass}"/>
-        <inertia ixx="${real_wheel_mass / 12.0 * (3*rear_wheel_radius + rear_wheel_width*rear_wheel_width)}" ixy="0.0" ixz="0.0" iyy="${real_wheel_mass / 12.0 * rear_wheel_radius*rear_wheel_radius}" iyz="0.0" izz="${real_wheel_mass / 12.0 * rear_wheel_radius*rear_wheel_radius}"/>
-      </inertial>
+      <xacro:cylinder_inertia m="${real_wheel_mass}" r="${rear_wheel_radius}" h="${rear_wheel_width}"/>
     </link>
     <!-- right wheel -->
@@ -133,9 +129,5 @@
         <material name="black"/>
       </visual>
-      <inertial>
-        <origin xyz="0 0 0" rpy="${PI/2} 0 0"/>
-        <mass value="${real_wheel_mass}"/>
-        <inertia ixx="${real_wheel_mass / 12.0 * (3*rear_wheel_radius + rear_wheel_width*rear_wheel_width)}" ixy="0.0" ixz="0.0" iyy="${real_wheel_mass / 12.0 * rear_wheel_radius*rear_wheel_radius}" iyz="0.0" izz="${real_wheel_mass / 12.0 * rear_wheel_radius*rear_wheel_radius}"/>
-      </inertial>
+      <xacro:cylinder_inertia m="${real_wheel_mass}" r="${rear_wheel_radius}" h="${rear_wheel_width}"/>
     </link>
     <!-- lidar -->

Commit message: Added imu link

File: ros/src/rosbot_description/urdf/rosbot.urdf.xacro (robot description, xacro)
@@ -24,4 +24,6 @@
     <xacro:property name="rear_wheel_axis_offset" value="0.1" />
     <xacro:property name="rear_wheel_distance" value="0.241" />
+    <!-- imu properties -->
+    <xacro:property name="imu_size" value="0.01" />
     <!-- PHYSICAL ROBOT MEASUREMENTS -->
     <!-- robot is 300mm wide, 460mm long, 170mm tall -->
@@ -148,4 +150,26 @@
       </visual>
     </link>
+    <!-- imu -->
+    <joint name="imu_joint" type="fixed">
+      <parent link="base_link"/>
+      <child link="imu_link"/>
+      <origin xyz="0 0 ${body_height + imu_size / 2}" rpy="0 0 ${PI}"/>
+      <axis xyz="0 0 1"/>
+    </joint>
+    <link name="imu_link">
+      <visual>
+        <origin xyz="0 0 0" rpy="0 0 0"/>
+        <geometry>
+          <box size="${imu_size} ${imu_size} ${imu_size}"/>
+        </geometry>
+        <material name="red"/>
+      </visual>
+      <collision>
+        <geometry>
+          <box size="${imu_size} ${imu_size} ${imu_size}"/>
+        </geometry>
+      </collision>
+      <xacro:box_inertia m="0.01" w="${imu_size}" d="${imu_size}" h="${imu_size}"/>
+    </link>
   </xacro:macro>
 </robot>

Commit message: Improved imu urdf

File: ros/src/rosbot_description/urdf/rosbot.urdf.xacro (robot description, xacro)
@@ -25,5 +25,5 @@
     <xacro:property name="rear_wheel_distance" value="0.241" />
     <!-- imu properties -->
-    <xacro:property name="imu_size" value="0.01" />
+    <xacro:property name="imu_size" value="0.05" />
     <!-- PHYSICAL ROBOT MEASUREMENTS -->
     <!-- robot is 300mm wide, 460mm long, 170mm tall -->
@@ -168,7 +168,8 @@
         <geometry>
           <box size="${imu_size} ${imu_size} ${imu_size}"/>
+          <cylinder length="${imu_size}" radius="${imu_size / 2}"/>
         </geometry>
       </collision>
-      <xacro:box_inertia m="0.01" w="${imu_size}" d="${imu_size}" h="${imu_size}"/>
+      <xacro:cylinder_inertia m="0.01" r="${imu_size}" h="${imu_size}"/>
     </link>
   </xacro:macro>
