Commit message: Added ekf and nav2_params configs, renamed rosbot links

File: ros/src/rosbot_description/urdf/rosbot_links.urdf.xacro (robot description, xacro)
@@ -5,5 +5,5 @@
   <!-- include inertia calculation macros -->
   <xacro:include filename="$(find rosbot_description)/urdf/inertia.urdf.xacro" />
-  <xacro:macro name="rosbot" params="prefix">
+  <xacro:macro name="rosbot_links" params="prefix">
     <!-- constants -->
     <xacro:property name="PI" value="3.1415926535897931"/>

File: ros/src/rosbot_description/urdf/rosbot_system.urdf.xacro (robot description, xacro)
@@ -1,13 +1,13 @@
 <?xml version="1.0"?>
-<robot xmlns:xacro="http://www.ros.org/wiki/xacro" name="diffdrive_robot">
+<robot xmlns:xacro="http://www.ros.org/wiki/xacro" name="rosbot">
   <xacro:arg name="use_sim" default="false" />
   <xacro:arg name="use_fake_hardware" default="false" />
   <xacro:arg name="fake_sensor_commands" default="false" />
   <xacro:arg name="prefix" default="" />
-  <xacro:include filename="$(find rosbot_description)/urdf/rosbot.urdf.xacro" />
+  <xacro:include filename="$(find rosbot_description)/urdf/rosbot_links.urdf.xacro" />
   <xacro:include filename="$(find rosbot_description)/gazebo/rosbot.gazebo.xacro" />
   <xacro:include filename="$(find rosbot_description)/gazebo/rosbot.materials.xacro" />
   <xacro:include filename="$(find rosbot_description)/ros2_control/rosbot_system.ros2_control.xacro" />
-  <xacro:rosbot prefix="$(arg prefix)" />
+  <xacro:rosbot_links prefix="$(arg prefix)" />
   <xacro:rosbot_gazebo prefix="$(arg prefix)" />
   <xacro:rosbot_system name="RosbotSystem" prefix="$(arg prefix)" use_fake_hardware="$(arg use_fake_hardware)" fake_sensor_commands="$(arg fake_sensor_commands)"/>

Commit message: Changed base link and footprint parent-child relationship

File: ros/src/rosbot_description/urdf/rosbot_links.urdf.xacro (robot description, xacro)
@@ -42,6 +42,6 @@
     <!-- base link -->
     <joint name="${prefix}base_joint" type="fixed">
-      <parent link="${prefix}base_footprint"/>
-      <child link="${prefix}base_link" />
+      <parent link="${prefix}base_link"/>
+      <child link="${prefix}base_bootprint" />
       <origin xyz="0 0 ${body_ground_offset}" rpy="0 0 0"/>
     </joint>

Commit message: Fixed typo

File: ros/src/rosbot_description/urdf/rosbot_links.urdf.xacro (robot description, xacro)
@@ -43,5 +43,5 @@
     <joint name="${prefix}base_joint" type="fixed">
       <parent link="${prefix}base_link"/>
-      <child link="${prefix}base_bootprint" />
+      <child link="${prefix}base_footprint" />
       <origin xyz="0 0 ${body_ground_offset}" rpy="0 0 0"/>
     </joint>

Commit message: Working on robot urdf

File: ros/src/rosbot_description/urdf/rosbot_links.urdf.xacro (robot description, xacro)
@@ -38,15 +38,8 @@
     <!-- large wheel pulley has 72 teeth -->
     <!-- motor to wheel gear ratio is 72/16 = 4.5 -->
-    <!-- base footprint -->
-    <link name="base_footprint"/>
-    <!-- base link -->
-    <joint name="${prefix}base_joint" type="fixed">
-      <parent link="${prefix}base_link"/>
-      <child link="${prefix}base_footprint" />
-      <origin xyz="0 0 ${body_ground_offset}" rpy="0 0 0"/>
-    </joint>
+    <!-- base link and footprint -->
     <link name="${prefix}base_link">
       <collision>
-        <origin xyz="${rear_wheel_axis_offset} 0 ${body_height/2}" rpy="0 0 0"/>
+        <origin xyz="${rear_wheel_axis_offset} 0 ${rear_wheel_ground_offset + body_height/2}" rpy="0 0 0"/>
         <geometry>
           <box size="${body_width} ${body_length} ${body_height}"/>
@@ -54,5 +47,5 @@
       </collision>
       <visual>
-        <origin xyz="${rear_wheel_axis_offset} 0 ${body_height/2}" rpy="0 0 0"/>
+        <origin xyz="${rear_wheel_axis_offset} 0 ${rear_wheel_ground_offset + body_height/2}" rpy="0 0 0"/>
         <geometry>
           <box size="${body_width} ${body_length} ${body_height}"/>
@@ -64,25 +57,10 @@
       <xacro:box_inertia m="${body_mass}" w="${body_width}" d="${body_length}" h="${body_height}"/>
     </link>
-    <!-- body -->
-    <!-- <joint name="${prefix}body_joint" type="fixed">
+    <link name="base_footprint"/>
+    <joint name="${prefix}base_joint" type="fixed">
       <parent link="${prefix}base_link"/>
-      <child link="${prefix}body"/>
-      <origin xyz="0 0 ${body_height + body_ground_offset + lidar_height / 2}" rpy="0 0 0"/>
-      <axis xyz="0 0 1"/>
+      <child link="${prefix}base_footprint" />
+      <origin xyz="${-rear_wheel_axis_offset} 0 0" rpy="0 0 0"/>
     </joint>
-    <link name="${prefix}body">
-      <visual>
-        <origin xyz="0 0 ${body_height + body_ground_offset + lidar_height / 2}" rpy="0 0 0"/>
-        <geometry>
-          <box size="${lidar_width} ${lidar_length} ${lidar_height}"/>
-        </geometry>
-        <material name="green"/>
-      </visual>
-      <inertial>
-        <origin xyz="${rear_wheel_axis_offset} 0 ${body_height/2 + body_ground_offset}" rpy="0 0 0"/>
-        <mass value="${body_mass}"/>
-        <inertia ixx="${body_mass / 12.0 * (body_length*body_length + body_height*body_height)}" ixy="0.0" ixz="0.0" iyy="${body_mass / 12.0 * (body_height*body_height + body_width*body_width)}" iyz="0.0" izz="${body_mass / 12.0 * (body_width*body_width + body_length*body_length)}"/>
-      </inertial>
-    </link> -->
     <!-- left wheel -->
     <joint name="${prefix}left_wheel_joint" type="continuous">

Commit message: Urdf 2

File: ros/src/rosbot_description/urdf/rosbot_links.urdf.xacro (robot description, xacro)
@@ -41,5 +41,5 @@
     <link name="${prefix}base_link">
       <collision>
-        <origin xyz="${rear_wheel_axis_offset} 0 ${rear_wheel_ground_offset + body_height/2}" rpy="0 0 0"/>
+        <origin xyz="${rear_wheel_axis_offset} 0 ${body_ground_offset + body_height/2}" rpy="0 0 0"/>
         <geometry>
           <box size="${body_width} ${body_length} ${body_height}"/>
@@ -47,5 +47,5 @@
       </collision>
       <visual>
-        <origin xyz="${rear_wheel_axis_offset} 0 ${rear_wheel_ground_offset + body_height/2}" rpy="0 0 0"/>
+        <origin xyz="${rear_wheel_axis_offset} 0 ${body_ground_offset + body_height/2}" rpy="0 0 0"/>
         <geometry>
           <box size="${body_width} ${body_length} ${body_height}"/>
@@ -61,5 +61,5 @@
       <parent link="${prefix}base_link"/>
       <child link="${prefix}base_footprint" />
-      <origin xyz="${-rear_wheel_axis_offset} 0 0" rpy="0 0 0"/>
+      <origin xyz="${rear_wheel_axis_offset} 0 0" rpy="0 0 0"/>
     </joint>
     <!-- left wheel -->
@@ -67,5 +67,5 @@
       <parent link="${prefix}base_link"/>
       <child link="${prefix}left_wheel"/>
-      <origin xyz="0 -${rear_wheel_distance/2} ${rear_wheel_ground_offset - body_ground_offset}" rpy="0 0 0"/>
+      <origin xyz="0 -${rear_wheel_distance/2} ${rear_wheel_ground_offset}" rpy="0 0 0"/>
       <axis xyz="0 1 0"/>
       <dynamics damping="0.2"/>
@@ -91,5 +91,5 @@
       <parent link="${prefix}base_link"/>
       <child link="${prefix}right_wheel"/>
-      <origin xyz="0 ${rear_wheel_distance/2} ${rear_wheel_ground_offset - body_ground_offset}" rpy="0 0 0"/>
+      <origin xyz="0 ${rear_wheel_distance/2} ${rear_wheel_ground_offset}" rpy="0 0 0"/>
       <axis xyz="0 1 0"/>
       <dynamics damping="0.2"/>

Commit message: Urdf 3

File: ros/src/rosbot_description/urdf/rosbot_links.urdf.xacro (robot description, xacro)
@@ -115,5 +115,5 @@
       <parent link="${prefix}base_link"/>
       <child link="${prefix}base_laser"/>
-      <origin xyz="${rear_wheel_axis_offset} 0 ${body_height + lidar_height / 2}" rpy="0 0 ${PI}"/>
+      <origin xyz="${rear_wheel_axis_offset} 0 ${body_ground_offset + body_height + lidar_height / 2}" rpy="0 0 ${PI}"/>
       <axis xyz="0 0 1"/>
     </joint>
@@ -132,5 +132,5 @@
       <parent link="base_link"/>
       <child link="imu_link"/>
-      <origin xyz="0 0 ${body_height + imu_size / 2}" rpy="0 0 ${PI}"/>
+      <origin xyz="0 0 ${body_ground_offset + body_height + imu_size / 2}" rpy="0 0 ${PI}"/>
       <axis xyz="0 0 1"/>
     </joint>

Commit message: Improved robot urdf formatting

File: ros/src/rosbot_description/urdf/rosbot_links.urdf.xacro (robot description, xacro)
@@ -64,11 +64,4 @@
     </joint>
     <!-- left wheel -->
-    <joint name="${prefix}left_wheel_joint" type="continuous">
-      <parent link="${prefix}base_link"/>
-      <child link="${prefix}left_wheel"/>
-      <origin xyz="0 -${rear_wheel_distance/2} ${rear_wheel_ground_offset}" rpy="0 0 0"/>
-      <axis xyz="0 1 0"/>
-      <dynamics damping="0.2"/>
-    </joint>
     <link name="${prefix}left_wheel">
       <collision>
@@ -87,12 +80,12 @@
       <xacro:cylinder_inertia m="${real_wheel_mass}" r="${rear_wheel_radius}" h="${rear_wheel_width}"/>
     </link>
-    <!-- right wheel -->
-    <joint name="${prefix}right_wheel_joint" type="continuous">
+    <joint name="${prefix}left_wheel_joint" type="continuous">
       <parent link="${prefix}base_link"/>
-      <child link="${prefix}right_wheel"/>
-      <origin xyz="0 ${rear_wheel_distance/2} ${rear_wheel_ground_offset}" rpy="0 0 0"/>
+      <child link="${prefix}left_wheel"/>
+      <origin xyz="0 -${rear_wheel_distance/2} ${rear_wheel_ground_offset}" rpy="0 0 0"/>
       <axis xyz="0 1 0"/>
       <dynamics damping="0.2"/>
     </joint>
+    <!-- right wheel -->
     <link name="${prefix}right_wheel">
       <collision>
@@ -111,11 +104,12 @@
       <xacro:cylinder_inertia m="${real_wheel_mass}" r="${rear_wheel_radius}" h="${rear_wheel_width}"/>
     </link>
+    <joint name="${prefix}right_wheel_joint" type="continuous">
+      <parent link="${prefix}base_link"/>
+      <child link="${prefix}right_wheel"/>
+      <origin xyz="0 ${rear_wheel_distance/2} ${rear_wheel_ground_offset}" rpy="0 0 0"/>
+      <axis xyz="0 1 0"/>
+      <dynamics damping="0.2"/>
+    </joint>
     <!-- lidar -->
-    <joint name="${prefix}lidar_joint" type="fixed">
-      <parent link="${prefix}base_link"/>
-      <child link="${prefix}base_laser"/>
-      <origin xyz="${rear_wheel_axis_offset} 0 ${body_ground_offset + body_height + lidar_height / 2}" rpy="0 0 ${PI}"/>
-      <axis xyz="0 0 1"/>
-    </joint>
     <link name="${prefix}base_laser">
       <visual>
@@ -128,11 +122,11 @@
       </visual>
     </link>
-    <!-- imu -->
-    <joint name="imu_joint" type="fixed">
-      <parent link="base_link"/>
-      <child link="imu_link"/>
-      <origin xyz="0 0 ${body_ground_offset + body_height + imu_size / 2}" rpy="0 0 ${PI}"/>
+    <joint name="${prefix}lidar_joint" type="fixed">
+      <parent link="${prefix}base_link"/>
+      <child link="${prefix}base_laser"/>
+      <origin xyz="${rear_wheel_axis_offset} 0 ${body_ground_offset + body_height + lidar_height / 2}" rpy="0 0 ${PI}"/>
       <axis xyz="0 0 1"/>
     </joint>
+    <!-- imu -->
     <link name="imu_link">
       <visual>
@@ -151,4 +145,10 @@
       <xacro:cylinder_inertia m="0.01" r="${imu_size}" h="${imu_size}"/>
     </link>
+    <joint name="imu_joint" type="fixed">
+      <parent link="base_link"/>
+      <child link="imu_link"/>
+      <origin xyz="0 0 ${body_ground_offset + body_height + imu_size / 2}" rpy="0 0 ${PI}"/>
+      <axis xyz="0 0 1"/>
+    </joint>
   </xacro:macro>
 </robot>

Commit message: Configured gazebo camera

File: ros/src/rosbot_description/urdf/rosbot_links.urdf.xacro (robot description, xacro)
@@ -30,5 +30,4 @@
     <xacro:property name="camera_length" value="0.05" />
     <xacro:property name="camera_height" value="0.025" />
-    <xacro:property name="camera_mass" value="0.05" />
     <!-- PHYSICAL ROBOT MEASUREMENTS -->
     <!-- robot is 300mm wide, 460mm long, 170mm tall -->
@@ -191,5 +190,5 @@
     <link name="${prefix}camera_link">
       <visual>
-        <origin xyz="0 0 0" rpy="0 0 0"/>
+        <origin xyz="${-camera_width / 2} 0 0" rpy="0 0 0"/>
         <geometry>
           <box size="${camera_width} ${camera_length} ${camera_height}"/>
@@ -197,16 +196,9 @@
         <material name="white"/>
       </visual>
-      <collision>
-        <origin xyz="0 0 0" rpy="0 0 0"/>
-        <geometry>
-          <box size="${camera_width} ${camera_length} ${camera_height}"/>
-        </geometry>
-      </collision>
-      <xacro:box_inertia m="${camera_mass}" w="${camera_width}" d="${camera_length}" h="${camera_height}"/>
     </link>
     <joint name="${prefix}camera_joint" type="fixed">
       <parent link="${prefix}body"/>
       <child link="${prefix}camera_link"/>
-      <origin xyz="${body_width / 2 - camera_width / 2} 0 ${body_height / 2 + camera_height / 2}" rpy="0 0 0"/>
+      <origin xyz="${body_width / 2} 0 ${body_height / 2 + camera_height / 2}" rpy="0 0 0"/>
       <axis xyz="0 0 1"/>
     </joint>
