Commit message: Improved gazebo configuration

File: ros/src/rosbot_description/gazebo/rosbot.gazebo.xacro (robot description, xacro)
@@ -2,72 +2,18 @@
 <robot xmlns:xacro="http://ros.org/wiki/xacro">
   <xacro:macro name="rosbot_gazebo" params="prefix">
-    <!-- Link1 -->
+    <!-- configure base link -->
     <gazebo reference="${prefix}base_link">
-      <material>Gazebo/Blue</material>
-    </gazebo>
-    <!-- Link2 -->
-    <gazebo reference="${prefix}link1">
+      <material>Gazebo/Orange</material>
+    </gazebo>
+    <!-- configure wheels -->
+    <gazebo reference="${prefix}left_wheel">
       <mu1>0.2</mu1>
       <mu2>0.2</mu2>
       <material>Gazebo/Black</material>
     </gazebo>
-    <!-- Link3 -->
-    <gazebo reference="${prefix}link2">
+    <gazebo reference="${prefix}right_wheel">
       <mu1>0.2</mu1>
       <mu2>0.2</mu2>
       <material>Gazebo/Black</material>
-    </gazebo>
-    <!-- camera_link -->
-    <gazebo reference="${prefix}camera_link">
-      <mu1>0.2</mu1>
-      <mu2>0.2</mu2>
-      <material>Gazebo/Red</material>
-    </gazebo>
-    <!-- camera -->
-    <gazebo reference="${prefix}camera_link">
-      <sensor type="camera" name="camera1">
-        <update_rate>30.0</update_rate>
-        <camera name="head">
-          <horizontal_fov>1.3962634</horizontal_fov>
-          <image>
-            <width>800</width>
-            <height>800</height>
-            <format>R8G8B8</format>
-          </image>
-          <clip>
-            <near>0.02</near>
-            <far>300</far>
-          </clip>
-          <noise>
-            <type>gaussian</type>
-            <!-- Noise is sampled independently per pixel on each frame.
-            That pixel's noise value is added to each of its color
-            channels, which at that point lie in the range [0,1]. -->
-            <mean>0.0</mean>
-            <stddev>0.007</stddev>
-          </noise>
-        </camera>
-        <plugin name="camera_controller" filename="libgazebo_ros_camera.so">
-          <alwaysOn>true</alwaysOn>
-          <updateRate>0.0</updateRate>
-          <cameraName>rosbot/camera1</cameraName>
-          <imageTopicName>image_raw</imageTopicName>
-          <cameraInfoTopicName>camera_info</cameraInfoTopicName>
-          <frameName>camera_link_optical</frameName>
-          <!-- setting hackBaseline to anything but 0.0 will cause a misalignment
-          between the gazebo sensor image and the frame it is supposed to
-          be attached to -->
-          <hackBaseline>0.0</hackBaseline>
-          <distortionK1>0.0</distortionK1>
-          <distortionK2>0.0</distortionK2>
-          <distortionK3>0.0</distortionK3>
-          <distortionT1>0.0</distortionT1>
-          <distortionT2>0.0</distortionT2>
-          <CxPrime>0</CxPrime>
-          <Cx>0.0</Cx>
-          <Cy>0.0</Cy>
-          <focalLength>0.0</focalLength>
-        </plugin>
-      </sensor>
     </gazebo>
     <!-- imu link -->
@@ -139,6 +85,8 @@
         </imu>
       </sensor>
+      <material>Gazebo/Red</material>
     </gazebo>
     <!-- differential drive -->
+    <!-- http://gazebosim.org/tutorials?tut=ros_gzplugins -->
     <gazebo>
       <plugin name='diff_drive' filename='libgazebo_ros_diff_drive.so'>
@@ -162,4 +110,15 @@
         <odometry_frame>odom</odometry_frame>
         <robot_base_frame>base_link</robot_base_frame>
+        <!-- use the same command topic as the real robot -->
+        <commandTopic>diff_drive_controller/cmd_vel_unstamped</commandTopic>
+        <!-- these are defaults -->
+        <!-- <odometryTopic>odom</odometryTopic> -->
+        <!-- <odometryFrame>odom</odometryFrame> -->
+        <!-- <robotBaseFrame>base_footprint</robotBaseFrame> -->
+        <!-- <odometrySource>1</odometrySource> -->
+        <!-- <publishOdom>true</publishOdom> -->
+        <!-- these default to false but had no effect -->
+        <!-- <publishWheelTF>true</publishWheelTF> -->
+        <!-- <publishWheelJointState>true</publishWheelJointState> -->
       </plugin>
     </gazebo>
@@ -198,4 +157,5 @@
         </plugin>
       </sensor>
+      <material>Gazebo/Green</material>
     </gazebo>
     <!-- TODO camera and depth sensing

File: ros/src/rosbot_description/urdf/rosbot.urdf.xacro (robot description, xacro)
@@ -2,11 +2,12 @@
 <robot name="rosbot"
   xmlns:xacro="http://www.ros.org/wiki/xacro">
-  <xacro:arg name="use_sim" default="false" />
+  <!-- TODO is use_sim argument used in any way? -->
+  <!-- <xacro:arg name="use_sim" default="false" /> -->
   <xacro:arg name="use_fake_hardware" default="false" />
   <xacro:arg name="fake_sensor_commands" default="false" />
   <xacro:arg name="prefix" default="" />
   <xacro:include filename="$(find rosbot_description)/urdf/rosbot_links.urdf.xacro" />
+  <xacro:include filename="$(find rosbot_description)/gazebo/rosbot.materials.xacro" />
   <xacro:include filename="$(find rosbot_description)/gazebo/rosbot.gazebo.xacro" />
-  <xacro:include filename="$(find rosbot_description)/gazebo/rosbot.materials.xacro" />
   <xacro:include filename="$(find rosbot_description)/ros2_control/rosbot_system.ros2_control.xacro" />
   <xacro:rosbot_links prefix="$(arg prefix)" />

Commit message: Configured robot inertia origin

File: ros/src/rosbot_description/gazebo/rosbot.gazebo.xacro (robot description, xacro)
@@ -22,5 +22,5 @@
         <plugin filename="libgazebo_ros_imu_sensor.so" name="imu_plugin">
           <ros>
-            <namespace>/demo</namespace>
+            <!-- <namespace>/demo</namespace> -->
             <remapping>~/out:=imu</remapping>
           </ros>
@@ -91,7 +91,7 @@
     <gazebo>
       <plugin name='diff_drive' filename='libgazebo_ros_diff_drive.so'>
-        <ros>
+        <!-- <ros>
           <namespace>/demo</namespace>
-        </ros>
+        </ros> -->
         <!-- wheels -->
         <left_joint>left_wheel_joint</left_joint>
@@ -111,5 +111,5 @@
         <robot_base_frame>base_link</robot_base_frame>
         <!-- use the same command topic as the real robot -->
-        <commandTopic>diff_drive_controller/cmd_vel_unstamped</commandTopic>
+        <!-- <commandTopic>/diff_drive_controller/cmd_vel_unstamped</commandTopic> -->
         <!-- these are defaults -->
         <!-- <odometryTopic>odom</odometryTopic> -->

File: ros/src/rosbot_description/urdf/inertia.urdf.xacro (robot description, xacro)
@@ -2,19 +2,19 @@
 <robot xmlns:xacro="http://www.ros.org/wiki/xacro">
     <!-- macros for calculating inertias of common 3d shapes  -->
-    <xacro:macro name="box_inertia" params="m w h d">
+    <xacro:macro name="box_inertia" params="m w h d originXYZ">
         <inertial>
-            <origin xyz="0 0 0" rpy="${pi/2} 0 ${pi/2}"/>
+            <origin xyz="${originXYZ}" rpy="${pi/2} 0 ${pi/2}"/>
             <mass value="${m}"/>
             <inertia ixx="${(m/12) * (h*h + d*d)}" ixy="0.0" ixz="0.0" iyy="${(m/12) * (w*w + d*d)}" iyz="0.0" izz="${(m/12) * (w*w + h*h)}"/>
         </inertial>
     </xacro:macro>
-    <xacro:macro name="cylinder_inertia" params="m r h">
+    <xacro:macro name="cylinder_inertia" params="m r h originXYZ">
         <inertial>
-            <origin xyz="0 0 0" rpy="${pi/2} 0 0" />
+            <origin xyz="${originXYZ}" rpy="${pi/2} 0 0" />
             <mass value="${m}"/>
             <inertia ixx="${(m/12) * (3*r*r + h*h)}" ixy = "0" ixz = "0" iyy="${(m/12) * (3*r*r + h*h)}" iyz = "0" izz="${(m/2) * (r*r)}"/>
         </inertial>
     </xacro:macro>
-    <xacro:macro name="sphere_inertia" params="m r">
+    <xacro:macro name="sphere_inertia" params="m r originXYZ">
         <inertial>
             <mass value="${m}"/>

File: ros/src/rosbot_description/urdf/rosbot_links.urdf.xacro (robot description, xacro)
@@ -53,5 +53,5 @@
         <material name="orange"/>
       </visual>
-      <xacro:box_inertia m="${body_mass}" w="${body_width}" d="${body_length}" h="${body_height}"/>
+      <xacro:box_inertia originXYZ="${rear_wheel_axis_offset} 0 ${body_ground_offset + body_height/2}" m="${body_mass}" w="${body_width}" d="${body_length}" h="${body_height}"/>
     </link>
     <link name="base_footprint"/>

Commit message: Working on gazebo simulation

File: ros/src/rosbot_description/gazebo/rosbot.gazebo.xacro (robot description, xacro)
@@ -6,14 +6,20 @@
       <material>Gazebo/Orange</material>
     </gazebo>
-    <!-- configure wheels -->
+    <!-- configure rear wheels -->
     <gazebo reference="${prefix}left_wheel">
-      <mu1>0.2</mu1>
-      <mu2>0.2</mu2>
+      <mu>0.6</mu>
+      <mu2>0.6</mu2>
       <material>Gazebo/Black</material>
     </gazebo>
     <gazebo reference="${prefix}right_wheel">
-      <mu1>0.2</mu1>
-      <mu2>0.2</mu2>
+      <mu>0.6</mu>
+      <mu2>0.6</mu2>
       <material>Gazebo/Black</material>
+    </gazebo>
+    <!-- configure caster wheel (use no friction) -->
+    <gazebo reference="${prefix}front_wheel">
+      <mu>0.0001</mu>
+      <mu2>0.0001</mu2>
+      <material>Gazebo/White</material>
     </gazebo>
     <!-- imu link -->
@@ -102,6 +108,6 @@
         <wheel_diameter>0.195</wheel_diameter>
         <!-- limits -->
-        <max_wheel_torque>20</max_wheel_torque>
-        <max_wheel_acceleration>1.0</max_wheel_acceleration>
+        <max_wheel_torque>50</max_wheel_torque>
+        <max_wheel_acceleration>2.0</max_wheel_acceleration>
         <!-- output -->
         <publish_odom>true</publish_odom>

File: ros/src/rosbot_description/urdf/inertia.urdf.xacro (robot description, xacro)
@@ -2,5 +2,5 @@
 <robot xmlns:xacro="http://www.ros.org/wiki/xacro">
     <!-- macros for calculating inertias of common 3d shapes  -->
-    <xacro:macro name="box_inertia" params="m w h d originXYZ">
+    <xacro:macro name="box_inertia" params="m w h d originXYZ:='0 0 0'">
         <inertial>
             <origin xyz="${originXYZ}" rpy="${pi/2} 0 ${pi/2}"/>
@@ -9,5 +9,5 @@
         </inertial>
     </xacro:macro>
-    <xacro:macro name="cylinder_inertia" params="m r h originXYZ">
+    <xacro:macro name="cylinder_inertia" params="m r h originXYZ:='0 0 0'">
         <inertial>
             <origin xyz="${originXYZ}" rpy="${pi/2} 0 0" />
@@ -16,5 +16,5 @@
         </inertial>
     </xacro:macro>
-    <xacro:macro name="sphere_inertia" params="m r originXYZ">
+    <xacro:macro name="sphere_inertia" params="m r">
         <inertial>
             <mass value="${m}"/>

File: ros/src/rosbot_description/urdf/rosbot_links.urdf.xacro (robot description, xacro)
@@ -4,6 +4,4 @@
   <xacro:include filename="$(find rosbot_description)/urdf/inertia.urdf.xacro" />
   <xacro:macro name="rosbot_links" params="prefix">
-    <!-- constants -->
-    <xacro:property name="PI" value="3.1415926535897931"/>
     <!-- body properties -->
     <xacro:property name="body_mass" value="6.0" />
@@ -16,10 +14,14 @@
     <xacro:property name="lidar_radius" value="0.0275" />
     <!-- rear wheel properties -->
-    <xacro:property name="real_wheel_mass" value="0.5" />
+    <xacro:property name="rear_wheel_mass" value="0.5" />
     <xacro:property name="rear_wheel_width" value="0.05" />
     <xacro:property name="rear_wheel_radius" value="0.0975" />
-    <xacro:property name="rear_wheel_ground_offset" value="0.0975" />
-    <xacro:property name="rear_wheel_axis_offset" value="0.1" />
+    <xacro:property name="rear_wheel_origin_x" value="-0.1" />
     <xacro:property name="rear_wheel_distance" value="0.241" />
+    <!-- front caster wheel properties -->
+    <xacro:property name="front_wheel_mass" value="0.2" />
+    <xacro:property name="front_wheel_width" value="0.025" />
+    <xacro:property name="front_wheel_radius" value="0.0385" />
+    <xacro:property name="front_wheel_origin_x" value="0.26757" />
     <!-- imu properties -->
     <xacro:property name="imu_size" value="0.02" />
@@ -31,5 +33,5 @@
     <!-- robot rear wheels axis is 97.5mm off the ground surface -->
     <!-- robot rear wheels axis is 100mm from the center of the body -->
-    <!-- front wheel radius 77mm  -->
+    <!-- front wheel diameter 77mm (radius 38.5mm)  -->
     <!-- robot front wheels axis is -267.57mm from the center of the body -->
     <!-- small motor pulley has 16 teeth -->
@@ -39,5 +41,5 @@
     <link name="${prefix}base_link">
       <collision>
-        <origin xyz="${rear_wheel_axis_offset} 0 ${body_ground_offset + body_height/2}" rpy="0 0 0"/>
+        <origin xyz="${rear_wheel_origin_x * -1} 0 ${body_ground_offset + body_height/2}" rpy="0 0 0"/>
         <geometry>
           <box size="${body_width} ${body_length} ${body_height}"/>
@@ -45,5 +47,5 @@
       </collision>
       <visual>
-        <origin xyz="${rear_wheel_axis_offset} 0 ${body_ground_offset + body_height/2}" rpy="0 0 0"/>
+        <origin xyz="${rear_wheel_origin_x * -1} 0 ${body_ground_offset + body_height/2}" rpy="0 0 0"/>
         <geometry>
           <box size="${body_width} ${body_length} ${body_height}"/>
@@ -53,5 +55,5 @@
         <material name="orange"/>
       </visual>
-      <xacro:box_inertia originXYZ="${rear_wheel_axis_offset} 0 ${body_ground_offset + body_height/2}" m="${body_mass}" w="${body_width}" d="${body_length}" h="${body_height}"/>
+      <xacro:box_inertia originXYZ="${rear_wheel_origin_x * -1} 0 ${body_ground_offset + body_height/2}" m="${body_mass}" w="${body_width}" d="${body_length}" h="${body_height}"/>
     </link>
     <link name="base_footprint"/>
@@ -59,16 +61,16 @@
       <parent link="${prefix}base_link"/>
       <child link="${prefix}base_footprint" />
-      <origin xyz="${rear_wheel_axis_offset} 0 0" rpy="0 0 0"/>
+      <origin xyz="${rear_wheel_origin_x * -1} 0 0" rpy="0 0 0"/>
     </joint>
     <!-- left wheel -->
     <link name="${prefix}left_wheel">
       <collision>
-        <origin xyz="0 0 0" rpy="${PI/2} 0 0"/>
-        <geometry>
-          <cylinder length="${rear_wheel_width}" radius="${rear_wheel_radius}"/>
-        </geometry>
-      </collision>
-      <visual>
-        <origin xyz="0 0 0" rpy="${PI/2} 0 0"/>
+        <origin xyz="0 0 0" rpy="${pi/2} 0 0"/>
+        <geometry>
+          <cylinder length="${rear_wheel_width}" radius="${rear_wheel_radius}"/>
+        </geometry>
+      </collision>
+      <visual>
+        <origin xyz="0 0 0" rpy="${pi/2} 0 0"/>
         <geometry>
           <cylinder length="${rear_wheel_width}" radius="${rear_wheel_radius}"/>
@@ -76,10 +78,10 @@
         <material name="black"/>
       </visual>
-      <xacro:cylinder_inertia m="${real_wheel_mass}" r="${rear_wheel_radius}" h="${rear_wheel_width}"/>
+      <xacro:cylinder_inertia m="${rear_wheel_mass}" r="${rear_wheel_radius}" h="${rear_wheel_width}"/>
     </link>
     <joint name="${prefix}left_wheel_joint" type="continuous">
       <parent link="${prefix}base_link"/>
       <child link="${prefix}left_wheel"/>
-      <origin xyz="0 -${rear_wheel_distance/2} ${rear_wheel_ground_offset}" rpy="0 0 0"/>
+      <origin xyz="0 -${rear_wheel_distance/2} ${rear_wheel_radius}" rpy="0 0 0"/>
       <axis xyz="0 1 0"/>
       <dynamics damping="0.2"/>
@@ -88,11 +90,11 @@
     <link name="${prefix}right_wheel">
       <collision>
-        <origin xyz="0 0 0" rpy="${PI/2} 0 0"/>
-        <geometry>
-          <cylinder length="${rear_wheel_width}" radius="${rear_wheel_radius}"/>
-        </geometry>
-      </collision>
-      <visual>
-        <origin xyz="0 0 0" rpy="${PI/2} 0 0"/>
+        <origin xyz="0 0 0" rpy="${pi/2} 0 0"/>
+        <geometry>
+          <cylinder length="${rear_wheel_width}" radius="${rear_wheel_radius}"/>
+        </geometry>
+      </collision>
+      <visual>
+        <origin xyz="0 0 0" rpy="${pi/2} 0 0"/>
         <geometry>
           <cylinder length="${rear_wheel_width}" radius="${rear_wheel_radius}"/>
@@ -100,13 +102,37 @@
         <material name="black"/>
       </visual>
-      <xacro:cylinder_inertia m="${real_wheel_mass}" r="${rear_wheel_radius}" h="${rear_wheel_width}"/>
+      <xacro:cylinder_inertia m="${rear_wheel_mass}" r="${rear_wheel_radius}" h="${rear_wheel_width}"/>
     </link>
     <joint name="${prefix}right_wheel_joint" type="continuous">
       <parent link="${prefix}base_link"/>
       <child link="${prefix}right_wheel"/>
-      <origin xyz="0 ${rear_wheel_distance/2} ${rear_wheel_ground_offset}" rpy="0 0 0"/>
+      <origin xyz="0 ${rear_wheel_distance/2} ${rear_wheel_radius}" rpy="0 0 0"/>
       <axis xyz="0 1 0"/>
       <dynamics damping="0.2"/>
     </joint>
+    <!-- front caster wheel -->
+    <link name="${prefix}front_wheel">
+      <collision>
+        <origin xyz="0 0 0" rpy="0 0 0"/>
+        <geometry>
+          <sphere radius="${front_wheel_radius}"/>
+        </geometry>
+      </collision>
+      <visual>
+        <origin xyz="0 0 0" rpy="0 0 0"/>
+        <geometry>
+          <sphere radius="${front_wheel_radius}"/>
+        </geometry>
+        <material name="white"/>
+      </visual>
+      <xacro:sphere_inertia m="${front_wheel_mass}" r="${front_wheel_radius}"/>
+    </link>
+    <joint name="${prefix}front_wheel_joint" type="fixed">
+      <parent link="${prefix}base_link"/>
+      <child link="${prefix}front_wheel"/>
+      <origin xyz="${front_wheel_origin_x - rear_wheel_origin_x} 0 ${front_wheel_radius}" rpy="0 0 0"/>
+      <axis xyz="0 0 1"/>
+      <dynamics damping="0.2"/>
+    </joint>
     <!-- lidar -->
     <link name="${prefix}base_laser">
@@ -123,5 +149,5 @@
       <parent link="${prefix}base_link"/>
       <child link="${prefix}base_laser"/>
-      <origin xyz="${rear_wheel_axis_offset} 0 ${body_ground_offset + body_height + lidar_height / 2}" rpy="0 0 ${PI}"/>
+      <origin xyz="${rear_wheel_origin_x * -1} 0 ${body_ground_offset + body_height + lidar_height / 2}" rpy="0 0 ${pi}"/>
       <axis xyz="0 0 1"/>
     </joint>
@@ -146,5 +172,5 @@
       <parent link="base_link"/>
       <child link="imu_link"/>
-      <origin xyz="0 0 ${body_ground_offset + body_height + imu_size / 2}" rpy="0 0 ${PI}"/>
+      <origin xyz="0 0 ${body_ground_offset + body_height + imu_size / 2}" rpy="0 0 0"/>
       <axis xyz="0 0 1"/>
     </joint>
