Commit message: Added body link

File: ros/src/rosbot_description/gazebo/rosbot.gazebo.xacro (robot description, xacro)
@@ -3,15 +3,15 @@
   <xacro:macro name="rosbot_gazebo" params="prefix">
     <!-- configure base link -->
-    <gazebo reference="${prefix}base_link">
+    <gazebo reference="${prefix}body">
       <material>Gazebo/Orange</material>
     </gazebo>
     <!-- configure rear wheels -->
     <gazebo reference="${prefix}left_wheel">
-      <mu>0.6</mu>
+      <mu1>0.6</mu1>
       <mu2>0.6</mu2>
       <material>Gazebo/Black</material>
     </gazebo>
     <gazebo reference="${prefix}right_wheel">
-      <mu>0.6</mu>
+      <mu1>0.6</mu1>
       <mu2>0.6</mu2>
       <material>Gazebo/Black</material>
@@ -19,6 +19,6 @@
     <!-- configure caster wheel (use no friction) -->
     <gazebo reference="${prefix}front_wheel">
-      <mu>0.0001</mu>
-      <mu2>0.0001</mu2>
+      <mu1>0</mu1>
+      <mu2>0</mu2>
       <material>Gazebo/White</material>
     </gazebo>
@@ -134,10 +134,10 @@
         <always_on>true</always_on>
         <visualize>true</visualize>
-        <update_rate>5</update_rate>
+        <update_rate>10</update_rate>
         <ray>
           <scan>
             <horizontal>
-              <samples>360</samples>
-              <resolution>1.000000</resolution>
+              <samples>920</samples>
+              <resolution>0.391</resolution>
               <min_angle>0.000000</min_angle>
               <max_angle>6.280000</max_angle>
@@ -146,6 +146,6 @@
           <range>
             <min>0.120000</min>
-            <max>3.5</max>
-            <resolution>0.015000</resolution>
+            <max>10</max>
+            <resolution>0.03</resolution>
           </range>
           <noise>

File: ros/src/rosbot_description/urdf/rosbot_links.urdf.xacro (robot description, xacro)
@@ -39,7 +39,16 @@
     <!-- motor to wheel gear ratio is 72/16 = 4.5 -->
     <!-- base link and footprint -->
-    <link name="${prefix}base_link">
-      <collision>
-        <origin xyz="${rear_wheel_origin_x * -1} 0 ${body_ground_offset + body_height/2}" rpy="0 0 0"/>
+    <link name="${prefix}base_link"/>
+    <!-- center of the robot projected on the ground, used for navigation calculation -->
+    <link name="base_footprint"/>
+    <joint name="${prefix}base_joint" type="fixed">
+      <parent link="${prefix}base_link"/>
+      <child link="${prefix}base_footprint" />
+      <origin xyz="${rear_wheel_origin_x * -1} 0 0" rpy="0 0 0"/>
+    </joint>
+    <!-- body -->
+    <link name="${prefix}body">
+      <collision>
+        <origin xyz="0 0 0" rpy="0 0 0"/>
         <geometry>
           <box size="${body_width} ${body_length} ${body_height}"/>
@@ -47,5 +56,5 @@
       </collision>
       <visual>
-        <origin xyz="${rear_wheel_origin_x * -1} 0 ${body_ground_offset + body_height/2}" rpy="0 0 0"/>
+        <origin xyz="0 0 0" rpy="0 0 0"/>
         <geometry>
           <box size="${body_width} ${body_length} ${body_height}"/>
@@ -55,11 +64,11 @@
         <material name="orange"/>
       </visual>
-      <xacro:box_inertia originXYZ="${rear_wheel_origin_x * -1} 0 ${body_ground_offset + body_height/2}" m="${body_mass}" w="${body_width}" d="${body_length}" h="${body_height}"/>
-    </link>
-    <link name="base_footprint"/>
-    <joint name="${prefix}base_joint" type="fixed">
-      <parent link="${prefix}base_link"/>
-      <child link="${prefix}base_footprint" />
-      <origin xyz="${rear_wheel_origin_x * -1} 0 0" rpy="0 0 0"/>
+      <xacro:box_inertia m="${body_mass}" w="${body_width}" d="${body_length}" h="${body_height}"/>
+    </link>
+    <joint name="${prefix}body_joint" type="fixed">
+      <parent link="${prefix}base_link"/>
+      <child link="${prefix}body"/>
+      <origin xyz="${-rear_wheel_origin_x} 0 ${body_ground_offset + body_height / 2}" rpy="0 0 0"/>
+      <axis xyz="0 0 1"/>
     </joint>
     <!-- left wheel -->
@@ -83,32 +92,32 @@
       <parent link="${prefix}base_link"/>
       <child link="${prefix}left_wheel"/>
+      <origin xyz="0 ${rear_wheel_distance/2} ${rear_wheel_radius}" rpy="0 0 0"/>
+      <axis xyz="0 1 0"/>
+      <dynamics damping="0.2"/>
+    </joint>
+    <!-- right wheel -->
+    <link name="${prefix}right_wheel">
+      <collision>
+        <origin xyz="0 0 0" rpy="${pi/2} 0 0"/>
+        <geometry>
+          <cylinder length="${rear_wheel_width}" radius="${rear_wheel_radius}"/>
+        </geometry>
+      </collision>
+      <visual>
+        <origin xyz="0 0 0" rpy="${pi/2} 0 0"/>
+        <geometry>
+          <cylinder length="${rear_wheel_width}" radius="${rear_wheel_radius}"/>
+        </geometry>
+        <material name="black"/>
+      </visual>
+      <xacro:cylinder_inertia m="${rear_wheel_mass}" r="${rear_wheel_radius}" h="${rear_wheel_width}"/>
+    </link>
+    <joint name="${prefix}right_wheel_joint" type="continuous">
+      <parent link="${prefix}base_link"/>
+      <child link="${prefix}right_wheel"/>
       <origin xyz="0 -${rear_wheel_distance/2} ${rear_wheel_radius}" rpy="0 0 0"/>
       <axis xyz="0 1 0"/>
       <dynamics damping="0.2"/>
     </joint>
-    <!-- right wheel -->
-    <link name="${prefix}right_wheel">
-      <collision>
-        <origin xyz="0 0 0" rpy="${pi/2} 0 0"/>
-        <geometry>
-          <cylinder length="${rear_wheel_width}" radius="${rear_wheel_radius}"/>
-        </geometry>
-      </collision>
-      <visual>
-        <origin xyz="0 0 0" rpy="${pi/2} 0 0"/>
-        <geometry>
-          <cylinder length="${rear_wheel_width}" radius="${rear_wheel_radius}"/>
-        </geometry>
-        <material name="black"/>
-      </visual>
-      <xacro:cylinder_inertia m="${rear_wheel_mass}" r="${rear_wheel_radius}" h="${rear_wheel_width}"/>
-    </link>
-    <joint name="${prefix}right_wheel_joint" type="continuous">
-      <parent link="${prefix}base_link"/>
-      <child link="${prefix}right_wheel"/>
-      <origin xyz="0 ${rear_wheel_distance/2} ${rear_wheel_radius}" rpy="0 0 0"/>
-      <axis xyz="0 1 0"/>
-      <dynamics damping="0.2"/>
-    </joint>
     <!-- front caster wheel -->
     <link name="${prefix}front_wheel">
@@ -129,7 +138,7 @@
     </link>
     <joint name="${prefix}front_wheel_joint" type="fixed">
-      <parent link="${prefix}base_link"/>
+      <parent link="${prefix}body"/>
       <child link="${prefix}front_wheel"/>
-      <origin xyz="${front_wheel_origin_x - rear_wheel_origin_x} 0 ${front_wheel_radius}" rpy="0 0 0"/>
+      <origin xyz="${front_wheel_origin_x} 0 ${front_wheel_radius - body_height / 2 - body_ground_offset}" rpy="0 0 0"/>
       <axis xyz="0 0 1"/>
       <dynamics damping="0.2"/>
@@ -147,7 +156,7 @@
     </link>
     <joint name="${prefix}lidar_joint" type="fixed">
-      <parent link="${prefix}base_link"/>
+      <parent link="${prefix}body"/>
       <child link="${prefix}base_laser"/>
-      <origin xyz="${rear_wheel_origin_x * -1} 0 ${body_ground_offset + body_height + lidar_height / 2}" rpy="0 0 ${pi}"/>
+      <origin xyz="0 0 ${body_height / 2 + lidar_height / 2}" rpy="0 0 ${pi}"/>
       <axis xyz="0 0 1"/>
     </joint>
@@ -170,7 +179,7 @@
     </link>
     <joint name="imu_joint" type="fixed">
-      <parent link="base_link"/>
+      <parent link="body"/>
       <child link="imu_link"/>
-      <origin xyz="0 0 ${body_ground_offset + body_height + imu_size / 2}" rpy="0 0 0"/>
+      <origin xyz="${rear_wheel_origin_x} 0 ${body_height / 2 + imu_size / 2}" rpy="0 0 0"/>
       <axis xyz="0 0 1"/>
     </joint>

Commit message: Added camera link

File: ros/src/rosbot_description/gazebo/rosbot.gazebo.xacro (robot description, xacro)
@@ -166,7 +166,43 @@
       <material>Gazebo/Green</material>
     </gazebo>
-    <!-- TODO camera and depth sensing
+    <!-- rgb camera -->
     <gazebo reference="camera_link">
-      <sensor name="depth_camera" type="depth">
+      <material>Gazebo/White</material>
+      <sensor type="camera" name="front_camera">
+        <update_rate>30.0</update_rate>
+        <visualize>true</visualize>
+        <camera name="head">
+          <horizontal_fov>1.3962634</horizontal_fov>
+          <image>
+            <width>800</width>
+            <height>800</height>
+            <format>R8G8B8</format>
+          </image>
+          <clip>
+            <near>0.05</near>
+            <far>300</far>
+          </clip>
+          <!-- <noise>
+            <type>gaussian</type>
+            <mean>0.0</mean>
+            <stddev>0.007</stddev>
+          </noise> -->
+        </camera>
+        <plugin name="camera_controller" filename="libgazebo_ros_camera.so">
+          <alwaysOn>true</alwaysOn>
+          <updateRate>0.0</updateRate>
+          <cameraName>rosbot/front_camera</cameraName>
+          <imageTopicName>image_raw</imageTopicName>
+          <cameraInfoTopicName>camera_info</cameraInfoTopicName>
+          <frameName>camera_link</frameName>
+          <hackBaseline>0.07</hackBaseline>
+          <distortionK1>0.0</distortionK1>
+          <distortionK2>0.0</distortionK2>
+          <distortionK3>0.0</distortionK3>
+          <distortionT1>0.0</distortionT1>
+          <distortionT2>0.0</distortionT2>
+        </plugin>
+      </sensor>
+      <!-- <sensor name="depth_camera" type="depth">
         <visualize>true</visualize>
         <update_rate>30.0</update_rate>
@@ -187,5 +223,5 @@
           <alwaysOn>true</alwaysOn>
           <updateRate>0.0</updateRate>
-          <frameName>camera_depth_frame</frameName>
+          <frameName>camera_link</frameName>
           <pointCloudCutoff>0.5</pointCloudCutoff>
           <pointCloudCutoffMax>3.0</pointCloudCutoffMax>
@@ -201,7 +237,6 @@
           <hackBaseline>0</hackBaseline>
         </plugin>
-      </sensor>
-    </gazebo>
-    -->
+      </sensor> -->
+    </gazebo>
   </xacro:macro>
 </robot>

File: ros/src/rosbot_description/urdf/rosbot_links.urdf.xacro (robot description, xacro)
@@ -26,4 +26,9 @@
     <!-- imu properties -->
     <xacro:property name="imu_size" value="0.02" />
+    <!-- camera properties -->
+    <xacro:property name="camera_width" value="0.025" />
+    <xacro:property name="camera_length" value="0.05" />
+    <xacro:property name="camera_height" value="0.025" />
+    <xacro:property name="camera_mass" value="0.05" />
     <!-- PHYSICAL ROBOT MEASUREMENTS -->
     <!-- robot is 300mm wide, 460mm long, 170mm tall -->
@@ -49,10 +54,4 @@
     <!-- body -->
     <link name="${prefix}body">
-      <collision>
-        <origin xyz="0 0 0" rpy="0 0 0"/>
-        <geometry>
-          <box size="${body_width} ${body_length} ${body_height}"/>
-        </geometry>
-      </collision>
       <visual>
         <origin xyz="0 0 0" rpy="0 0 0"/>
@@ -64,4 +63,10 @@
         <material name="orange"/>
       </visual>
+      <collision>
+        <origin xyz="0 0 0" rpy="0 0 0"/>
+        <geometry>
+          <box size="${body_width} ${body_length} ${body_height}"/>
+        </geometry>
+      </collision>
       <xacro:box_inertia m="${body_mass}" w="${body_width}" d="${body_length}" h="${body_height}"/>
     </link>
@@ -74,10 +79,4 @@
     <!-- left wheel -->
     <link name="${prefix}left_wheel">
-      <collision>
-        <origin xyz="0 0 0" rpy="${pi/2} 0 0"/>
-        <geometry>
-          <cylinder length="${rear_wheel_width}" radius="${rear_wheel_radius}"/>
-        </geometry>
-      </collision>
       <visual>
         <origin xyz="0 0 0" rpy="${pi/2} 0 0"/>
@@ -87,4 +86,10 @@
         <material name="black"/>
       </visual>
+      <collision>
+        <origin xyz="0 0 0" rpy="${pi/2} 0 0"/>
+        <geometry>
+          <cylinder length="${rear_wheel_width}" radius="${rear_wheel_radius}"/>
+        </geometry>
+      </collision>
       <xacro:cylinder_inertia m="${rear_wheel_mass}" r="${rear_wheel_radius}" h="${rear_wheel_width}"/>
     </link>
@@ -98,10 +103,4 @@
     <!-- right wheel -->
     <link name="${prefix}right_wheel">
-      <collision>
-        <origin xyz="0 0 0" rpy="${pi/2} 0 0"/>
-        <geometry>
-          <cylinder length="${rear_wheel_width}" radius="${rear_wheel_radius}"/>
-        </geometry>
-      </collision>
       <visual>
         <origin xyz="0 0 0" rpy="${pi/2} 0 0"/>
@@ -111,4 +110,10 @@
         <material name="black"/>
       </visual>
+      <collision>
+        <origin xyz="0 0 0" rpy="${pi/2} 0 0"/>
+        <geometry>
+          <cylinder length="${rear_wheel_width}" radius="${rear_wheel_radius}"/>
+        </geometry>
+      </collision>
       <xacro:cylinder_inertia m="${rear_wheel_mass}" r="${rear_wheel_radius}" h="${rear_wheel_width}"/>
     </link>
@@ -122,17 +127,17 @@
     <!-- front caster wheel -->
     <link name="${prefix}front_wheel">
-      <collision>
+      <visual>
         <origin xyz="0 0 0" rpy="0 0 0"/>
         <geometry>
           <sphere radius="${front_wheel_radius}"/>
         </geometry>
-      </collision>
-      <visual>
+        <material name="white"/>
+      </visual>
+      <collision>
         <origin xyz="0 0 0" rpy="0 0 0"/>
         <geometry>
           <sphere radius="${front_wheel_radius}"/>
         </geometry>
-        <material name="white"/>
-      </visual>
+      </collision>
       <xacro:sphere_inertia m="${front_wheel_mass}" r="${front_wheel_radius}"/>
     </link>
@@ -149,5 +154,4 @@
         <origin xyz="0 0 0" rpy="0 0 0"/>
         <geometry>
-          <!-- <box size="${lidar_width} ${lidar_length} ${lidar_height}"/> -->
           <cylinder length="${lidar_height}" radius="${lidar_radius}"/>
         </geometry>
@@ -182,4 +186,27 @@
       <child link="imu_link"/>
       <origin xyz="${rear_wheel_origin_x} 0 ${body_height / 2 + imu_size / 2}" rpy="0 0 0"/>
+      <axis xyz="0 0 1"/>
+    </joint>
+    <!-- camera -->
+    <link name="${prefix}camera_link">
+      <visual>
+        <origin xyz="0 0 0" rpy="0 0 0"/>
+        <geometry>
+          <box size="${camera_width} ${camera_length} ${camera_height}"/>
+        </geometry>
+        <material name="white"/>
+      </visual>
+      <collision>
+        <origin xyz="0 0 0" rpy="0 0 0"/>
+        <geometry>
+          <box size="${camera_width} ${camera_length} ${camera_height}"/>
+        </geometry>
+      </collision>
+      <xacro:box_inertia m="${camera_mass}" w="${camera_width}" d="${camera_length}" h="${camera_height}"/>
+    </link>
+    <joint name="${prefix}camera_joint" type="fixed">
+      <parent link="${prefix}body"/>
+      <child link="${prefix}camera_link"/>
+      <origin xyz="${body_width / 2 - camera_width / 2} 0 ${body_height / 2 + camera_height / 2}" rpy="0 0 0"/>
       <axis xyz="0 0 1"/>
     </joint>

Commit message: Improved gazebo configuration

File: ros/src/rosbot_description/gazebo/rosbot.gazebo.xacro (robot description, xacro)
@@ -166,11 +166,11 @@
       <material>Gazebo/Green</material>
     </gazebo>
-    <!-- rgb camera -->
-    <gazebo reference="camera_link">
+    <!-- camera -->
+    <gazebo reference="rgb_camera_link">
       <material>Gazebo/White</material>
-      <sensor type="camera" name="front_camera">
+      <sensor type="camera" name="rgb_camera">
         <update_rate>30.0</update_rate>
         <visualize>true</visualize>
-        <camera name="head">
+        <camera name="rgb_camera">
           <horizontal_fov>1.3962634</horizontal_fov>
           <image>
@@ -189,11 +189,9 @@
           </noise>
         </camera>
-        <plugin name="front_camera_controller" filename="libgazebo_ros_camera.so">
+        <plugin name="rgb_camera_controller" filename="libgazebo_ros_camera.so">
+          <frameName>rgb_camera_link</frameName>
           <alwaysOn>true</alwaysOn>
           <updateRate>0.0</updateRate>
-          <cameraName>rosbot/front_camera</cameraName>
-          <imageTopicName>image_raw</imageTopicName>
-          <cameraInfoTopicName>camera_info</cameraInfoTopicName>
-          <frameName>camera_link</frameName>
+          <baseline>0.2</baseline>
           <hackBaseline>0.07</hackBaseline>
           <distortionK1>0.0</distortionK1>
@@ -202,12 +200,18 @@
           <distortionT1>0.0</distortionT1>
           <distortionT2>0.0</distortionT2>
+          <pointCloudCutoff>0.5</pointCloudCutoff>
+          <pointCloudCutoffMax>3.0</pointCloudCutoffMax>
+          <CxPrime>0</CxPrime>
+          <Cx>0</Cx>
+          <Cy>0</Cy>
         </plugin>
       </sensor>
     </gazebo>
     <!-- depth camera -->
-    <!-- <gazebo reference="camera_link">
+    <!-- <gazebo reference="rgb_camera_link">
       <sensor type="depth" name="depth_camera">
-        <update_rate>20</update_rate>
-        <camera>
+        <update_rate>30.0</update_rate>
+        <visualize>true</visualize>
+        <camera name="depth_camera">
           <horizontal_fov>1.047198</horizontal_fov>
           <image>
@@ -218,30 +222,28 @@
           <clip>
             <near>0.05</near>
-            <far>3</far>
+            <far>3.0</far>
           </clip>
+          <noise>
+            <type>gaussian</type>
+            <mean>0.0</mean>
+            <stddev>0.007</stddev>
+          </noise>
         </camera>
-        <plugin name="depth_camera_controller" filename="libgazebo_ros_openni_kinect.so">
+        <plugin name="depth_camera_controller" filename="libgazebo_ros_camera.so">
+          <frameName>depth_camera_link</frameName>
+          <alwaysOn>true</alwaysOn>
+          <updateRate>0.0</updateRate>
           <baseline>0.2</baseline>
-          <alwaysOn>true</alwaysOn>
-          <updateRate>1.0</updateRate>
-          <cameraName>depth_camera_ir</cameraName>
-          <imageTopicName>/depth_camera/color/image_raw</imageTopicName>
-          <cameraInfoTopicName>/depth_camera/color/camera_info</cameraInfoTopicName>
-          <depthImageTopicName>/depth_camera/depth/image_raw</depthImageTopicName>
-          <depthImageInfoTopicName>/depth_camera/depth/camera_info</depthImageInfoTopicName>
-          <pointCloudTopicName>/depth_camera/depth/points</pointCloudTopicName>
-          <frameName>camera_link</frameName>
+          <hackBaseline>0.07</hackBaseline>
+          <distortionK1>0.0</distortionK1>
+          <distortionK2>0.0</distortionK2>
+          <distortionK3>0.0</distortionK3>
+          <distortionT1>0.0</distortionT1>
+          <distortionT2>0.0</distortionT2>
           <pointCloudCutoff>0.5</pointCloudCutoff>
           <pointCloudCutoffMax>3.0</pointCloudCutoffMax>
-          <distortionK1>0.00000001</distortionK1>
-          <distortionK2>0.00000001</distortionK2>
-          <distortionK3>0.00000001</distortionK3>
-          <distortionT1>0.00000001</distortionT1>
-          <distortionT2>0.00000001</distortionT2>
           <CxPrime>0</CxPrime>
           <Cx>0</Cx>
           <Cy>0</Cy>
-          <focalLength>0</focalLength>
-          <hackBaseline>0</hackBaseline>
         </plugin>
       </sensor>

File: ros/src/rosbot_description/urdf/rosbot_links.urdf.xacro (robot description, xacro)
@@ -187,6 +187,6 @@
       <axis xyz="0 0 1"/>
     </joint>
-    <!-- camera -->
-    <link name="${prefix}camera_link">
+    <!-- rgb camera -->
+    <link name="${prefix}rgb_camera_link">
       <visual>
         <origin xyz="${-camera_width / 2} 0 0" rpy="0 0 0"/>
@@ -199,40 +199,14 @@
     <joint name="${prefix}camera_joint" type="fixed">
       <parent link="${prefix}body"/>
-      <child link="${prefix}camera_link"/>
+      <child link="${prefix}rgb_camera_link"/>
       <origin xyz="${body_width / 2} 0 ${body_height / 2 + camera_height / 2}" rpy="0 0 0"/>
-      <axis xyz="0 0 1"/>
-    </joint>
-    <!-- TODO camera and depth sensing
-    <link name="camera_link">
-      <visual>
-        <origin xyz="0 0 0" rpy="0 0 0"/>
-        <geometry>
-          <box size="0.015 0.130 0.022"/>
-        </geometry>
-      </visual>
-      <collision>
-        <origin xyz="0 0 0" rpy="0 0 0"/>
-        <geometry>
-          <box size="0.015 0.130 0.022"/>
-        </geometry>
-      </collision>
-      <inertial>
-        <origin xyz="0 0 0" rpy="0 0 0"/>
-        <mass value="0.035"/>
-        <inertia ixx="0.001" ixy="0" ixz="0" iyy="0.001" iyz="0" izz="0.001" />
-      </inertial>
-    </link>
-    <joint name="camera_joint" type="fixed">
-      <parent link="base_link"/>
-      <child link="camera_link"/>
-      <origin xyz="0.215 0 0.05" rpy="0 0 0"/>
-    </joint>
-    <link name="camera_depth_frame"/>
-    <joint name="camera_depth_joint" type="fixed">
-      <origin xyz="0 0 0" rpy="${-pi/2} 0 ${-pi}"/>
-      <parent link="camera_link"/>
-      <child link="camera_depth_frame"/>
-    </joint>
-    -->
+    </joint>
+    <!-- depth camera -->
+    <link name="depth_camera_link"/>
+    <joint name="depth_camera_joint" type="fixed">
+      <origin xyz="0 0 0" rpy="${-pi/2} 0 ${pi/2}"/>
+      <parent link="rgb_camera_link"/>
+      <child link="depth_camera_link"/>
+    </joint>
   </xacro:macro>
 </robot>
